Commit message: aligned differential module wheel joint axis

File: robotics/transbot-ros2ws/src/transbot_description/urdf/rigid_forklift/mobilebase/diff/diff.urdf.xacro (robot description, xacro)
@@ -63,5 +63,5 @@
             </joint>
             <joint name="${prefix}cj1" type="continuous">
-                <origin xyz="0.0 +0.280 0.0" rpy="+1.57 0.0 0.0"/>
+                <origin xyz="0.0 +0.280 0.0" rpy="-1.57 0.0 0.0"/>
                 <axis xyz="0.0 0.0 1.0"/>
                 <parent link="${prefix}_${suffix}"/>

Commit message: OpenSCAD to URDF + Gazebo exporter

File: robotics/transbot-ros2ws/src/transbot_description/urdf/rigid_forklift/mobilebase/diff/diff.urdf.xacro (robot description, xacro)
@@ -4,5 +4,5 @@
         <xacro:unless value="${use__all__}">
             <!-- ROOT LINK -->
-            <link name="${prefix}_${suffix}">
+            <link name="${prefix}_">
                 <inertial>
                     <origin xyz="1.2249181909870052e-11 1.8496264683903782e-09 -1.6256482632337307e-11" rpy="0.0 0.0 0.0"></origin>
