Commit message: basic manipulator teleop

File: robotics/transbot-ros2ws/src/transbot_description/urdf/rigid_forklift_dsusp_rr/mobilebase/doublebar/doublebar.urdf.xacro (robot description, xacro)
@@ -27,5 +27,5 @@
 			<parent link="${prefix}${name}${suffix}_"></parent>
 			<child link="${prefix}${name}${suffix}diff/_"></child>
-			<dynamics damping="10" friction="10"></dynamics>
+			<dynamics damping="1" friction="0"></dynamics>
 			<axis xyz="1 0 0"></axis>
 		</joint>

File: robotics/transbot-ros2ws/src/transbot_description/urdf/rigid_forklift_dsusp_rr/mobilebase/mobilebase.urdf.xacro (robot description, xacro)
@@ -16,5 +16,5 @@
 			<parent link="${prefix}${name}${suffix}_"></parent>
 			<child link="${prefix}${name}${suffix}doublebar/_"></child>
-			<dynamics damping="10" friction="10"></dynamics>
+			<dynamics damping="1" friction="0"></dynamics>
 			<axis xyz="0 1 0"></axis>
 		</joint>
