Commit message: SCAD Models

File: robotics/transbot-ros2ws/src/transbot_description/urdf/rigid_forklift_dsusp_rr/manipulator/manipulator.urdf.xacro (robot description, xacro)
@@ -16,8 +16,8 @@
 			<child link="${prefix}${name}${suffix}horquilla"></child>
 			<axis xyz="0 0 1"></axis>
-			<limit lower="-0.05" upper="1.77" effort="1000000.0" velocity="1000000.0"></limit>
+			<limit lower="0.0" upper="1.27" effort="1000000.0" velocity="1000000.0"></limit>
 		</joint>
 		<joint name="j/${prefix}${name}${suffix}unna0" type="prismatic">
-			<origin xyz="0.075 -0.05 -0.05" rpy="0.0 0.0 0.0"></origin>
+			<origin xyz="0.075 -0.05 -0.1" rpy="0.0 0.0 0.0"></origin>
 			<parent link="${prefix}${name}${suffix}horquilla"></parent>
 			<child link="${prefix}${name}${suffix}unna0"></child>
@@ -26,5 +26,5 @@
 		</joint>
 		<joint name="j/${prefix}${name}${suffix}unna1" type="prismatic">
-			<origin xyz="0.075 0.05 -0.05" rpy="0.0 0.0 0.0"></origin>
+			<origin xyz="0.075 0.05 -0.1" rpy="0.0 0.0 0.0"></origin>
 			<parent link="${prefix}${name}${suffix}horquilla"></parent>
 			<child link="${prefix}${name}${suffix}unna1"></child>

File: robotics/transbot-ros2ws/src/transbot_description/urdf/rigid_forklift_dsusp_rr/manipulator/portico.urdf.xacro (robot description, xacro)
@@ -4,7 +4,7 @@
 		<link name="${prefix}${name}${suffix}">
 			<inertial density="7850">
-				<origin xyz="1.6526583292160544e-10 3.3846442582344794e-07 1.02374387178426" rpy="0 0 0"></origin>
-				<mass value="1.834407603989045"></mass>
-				<inertia ixx="0.8985282082372781" ixy="-1.2126585762585642e-10" ixz="3.1036320912009606e-10" iyy="0.7266451146659652" iyz="3.872711657138292e-07" izz="0.1749404398043246"></inertia>
+				<origin xyz="0.0 0.0 0.7915687128154306" rpy="0 0 0"></origin>
+				<mass value="1.3944067371388276"></mass>
+				<inertia ixx="0.4245243160703809" ixy="-1.2126596023639044e-10" ixz="-0.0" iyy="0.29817981721229225" iyz="1.241763432820638e-07" izz="0.12866851005431576"></inertia>
 			</inertial>
 			<visual>

File: robotics/transbot-ros2ws/src/transbot_description/urdf/rigid_forklift_dsusp_rr/manipulator/unna.urdf.xacro (robot description, xacro)
@@ -4,7 +4,7 @@
 		<link name="${prefix}${name}${suffix}">
 			<inertial density="7850">
-				<origin xyz="0.31713588379419205 -3.2682716149784016e-10 0.0016358343282475052" rpy="0 0 0"></origin>
-				<mass value="0.2319000195711851"></mass>
-				<inertia ixx="0.00014810430585443694" ixy="-2.4036117171074392e-11" ixz="0.0002657068439596089" iyy="0.011016142898947569" iyz="-1.2398188787661524e-13" izz="0.011085444903884207"></inertia>
+				<origin xyz="0.19335801902328506 3.8987254598624655e-10 0.01535802775643009" rpy="0 0 0"></origin>
+				<mass value="0.19440000566343466"></mass>
+				<inertia ixx="0.0003702513319354325" ixy="1.465484115391557e-11" ixz="0.0006457186385303325" iyy="0.005511267229784068" iyz="2.76272489497312e-12" izz="0.005323265933474595"></inertia>
 			</inertial>
 			<visual>

File: robotics/transbot-ros2ws/src/transbot_description/urdf/rigid_forklift_dsusp_rr/mobilebase/castor/wheel.urdf.xacro (robot description, xacro)
@@ -4,7 +4,7 @@
 		<link name="${prefix}${name}${suffix}">
 			<inertial density="2500">
-				<origin xyz="-7.119797463040393e-10 -2.8817871019630973e-10 -1.3427359559848857e-10" rpy="0 0 0"></origin>
+				<origin xyz="-1.4410434099052077e-09 -9.755815930202686e-11 -1.3427359559848857e-10" rpy="0 0 0"></origin>
 				<mass value="0.49389696990450227"></mass>
-				<inertia ixx="0.0005393656238084077" ixy="-7.08692262715893e-13" ixz="-1.30266163501026e-12" iyy="0.0005393657450743677" iyz="1.181925119411268e-13" izz="0.0009120412869378921"></inertia>
+				<inertia ixx="0.0005393656844413878" ixy="-1.6560826089644183e-12" ixz="-1.3026615866607103e-12" iyy="0.000539365805707347" iyz="1.1819249929968234e-13" izz="0.0009120414082038515"></inertia>
 			</inertial>
 			<visual>

File: robotics/transbot-ros2ws/src/transbot_description/urdf/rigid_forklift_dsusp_rr/mobilebase/control.urdf.xacro (robot description, xacro)
@@ -3,8 +3,8 @@
 	<xacro:macro name="control" params="prefix='' name='control' suffix=''">
 		<link name="${prefix}${name}${suffix}">
-			<inertial density="7850">
-				<origin xyz="-0.11800876511481027 0.09354560312818934 0.10163800234275462" rpy="0 0 0"></origin>
-				<mass value="11.364147067070007"></mass>
-				<inertia ixx="0.20224443786592244" ixy="0.04016673361813658" ixz="0.03380698382561664" iyy="0.1792783009602844" iyz="-0.02783002652166694" izz="0.2541928858214154"></inertia>
+			<inertial density="13800">
+				<origin xyz="0.002084133424969194 -0.1180087385611795 0.10163798440735253" rpy="0 0 0"></origin>
+				<mass value="11.36414830883344"></mass>
+				<inertia ixx="0.1792783214037889" ixy="-0.005400248580619397" ixz="0.0018980197654414812" iyy="0.17123017326450496" iyz="0.033806977088390505" izz="0.2231786465435561"></inertia>
 			</inertial>
 			<visual>

File: robotics/transbot-ros2ws/src/transbot_description/urdf/rigid_forklift_dsusp_rr/mobilebase/doublebar/diff/wheel.urdf.xacro (robot description, xacro)
@@ -4,7 +4,7 @@
 		<link name="${prefix}${name}${suffix}">
 			<inertial density="2500">
-				<origin xyz="8.79249560971962e-12 -3.3967090836983846e-10 -2.110198946332709e-10" rpy="0 0 0"></origin>
+				<origin xyz="1.0821533058116455e-11 -3.3899456255370624e-10 -2.110198946332709e-10" rpy="0 0 0"></origin>
 				<mass value="0.437733872483174"></mass>
-				<inertia ixx="0.00046364856795359316" ixy="-4.0221587647650746e-12" ixz="-3.552713686922178e-13" iyy="0.0004636485679535932" iyz="4.626243025176925e-16" izz="0.0008105681748323452"></inertia>
+				<inertia ixx="0.00046364856795359316" ixy="-4.0216961721366314e-12" ixz="-3.552713688796411e-13" iyy="0.0004636485679535932" iyz="4.626242400432536e-16" izz="0.0008105681748323452"></inertia>
 			</inertial>
 			<visual>

File: robotics/transbot-ros2ws/src/transbot_description/urdf/rigid_forklift_dsusp_rr/mobilebase/doublebar/doublebar.urdf.xacro (robot description, xacro)
@@ -27,5 +27,5 @@
 			<parent link="${prefix}${name}${suffix}_"></parent>
 			<child link="${prefix}${name}${suffix}diff/_"></child>
-			<dynamics damping="1" friction="0"></dynamics>
+			<dynamics damping="10" friction="10"></dynamics>
 			<axis xyz="1 0 0"></axis>
 		</joint>

File: robotics/transbot-ros2ws/src/transbot_description/urdf/rigid_forklift_dsusp_rr/mobilebase/mobilebase.urdf.xacro (robot description, xacro)
@@ -16,5 +16,5 @@
 			<parent link="${prefix}${name}${suffix}_"></parent>
 			<child link="${prefix}${name}${suffix}doublebar/_"></child>
-			<dynamics damping="1" friction="0"></dynamics>
+			<dynamics damping="10" friction="10"></dynamics>
 			<axis xyz="0 1 0"></axis>
 		</joint>
@@ -30,9 +30,9 @@
 		</joint>
 		<joint name="j/${prefix}${name}${suffix}control" type="prismatic">
-			<origin xyz="0.0 0.0 0.17" rpy="0.0 0.0 0.0"></origin>
+			<origin xyz="0.075 0.0 0.17" rpy="0.0 0.0 1.5707963267948966"></origin>
 			<parent link="${prefix}${name}${suffix}_"></parent>
 			<child link="${prefix}${name}${suffix}control"></child>
 			<dynamics damping="10" friction="10"></dynamics>
-			<axis xyz="1 0 0"></axis>
+			<axis xyz="0 -1 0"></axis>
 			<limit lower="0.0" upper="0.5" effort="1000000.0" velocity="1000000.0"></limit>
 		</joint>
