Commit message: Actualizado SCAD2URDF (JAR XIII)
Actualización librería OpenSCAD to URDF. Agregado junta de revolución + extras para paper JAR XIII

File: robotics/transbot-ros2ws/src/transbot_description/urdf/rigid_forklift/manipulator/horquilla.urdf.xacro (robot description, xacro)
@@ -13,5 +13,5 @@
 				</geometry>
 				<material name="">
-					<color rgba="1 1 1 1"></color>
+					<color rgba="0.2 0.7 0.2 1"></color>
 				</material>
 			</visual>

File: robotics/transbot-ros2ws/src/transbot_description/urdf/rigid_forklift/manipulator/portico.urdf.xacro (robot description, xacro)
@@ -13,5 +13,5 @@
 				</geometry>
 				<material name="">
-					<color rgba="1 1 1 1"></color>
+					<color rgba="0.7 0.2 0.2 1"></color>
 				</material>
 			</visual>

File: robotics/transbot-ros2ws/src/transbot_description/urdf/rigid_forklift/manipulator/unna.urdf.xacro (robot description, xacro)
@@ -13,5 +13,5 @@
 				</geometry>
 				<material name="">
-					<color rgba="1 1 1 1"></color>
+					<color rgba="0.2 0.2 0.7 1"></color>
 				</material>
 			</visual>

File: robotics/transbot-ros2ws/src/transbot_description/urdf/rigid_forklift/mobilebase/castor/wheel.urdf.xacro (robot description, xacro)
@@ -4,7 +4,7 @@
 		<link name="${prefix}${name}${suffix}">
 			<inertial density="2500">
-				<origin xyz="-7.130287587696525e-10 -2.809854818606764e-10 -1.3427359559848857e-10" rpy="0 0 0"></origin>
+				<origin xyz="-1.4362479243481186e-09 -9.755815930202686e-11 -1.3427359559848857e-10" rpy="0 0 0"></origin>
 				<mass value="0.49389696990450227"></mass>
-				<inertia ixx="0.0005393656238084077" ixy="-7.086922650997735e-13" ixz="-1.3026616349406924e-12" iyy="0.0005393657450743677" iyz="1.1819251146409114e-13" izz="0.0009120412869378921"></inertia>
+				<inertia ixx="0.0005393656844413878" ixy="-1.6560826091954824e-12" ixz="-1.3026615869787342e-12" iyy="0.0005393658057073471" iyz="1.1819249929968234e-13" izz="0.0009120414082038516"></inertia>
 			</inertial>
 			<visual>
@@ -13,5 +13,5 @@
 				</geometry>
 				<material name="">
-					<color rgba="1 1 1 1"></color>
+					<color rgba="0.2 0.2 0.2 1"></color>
 				</material>
 			</visual>

File: robotics/transbot-ros2ws/src/transbot_description/urdf/rigid_forklift/mobilebase/chassis.urdf.xacro (robot description, xacro)
@@ -13,5 +13,5 @@
 				</geometry>
 				<material name="">
-					<color rgba="1 1 1 1"></color>
+					<color rgba="1 1 0 1"></color>
 				</material>
 			</visual>

File: robotics/transbot-ros2ws/src/transbot_description/urdf/rigid_forklift/mobilebase/control.urdf.xacro (robot description, xacro)
@@ -3,5 +3,5 @@
 	<xacro:macro name="control" params="prefix='' name='control' suffix=''">
 		<link name="${prefix}${name}${suffix}">
-			<inertial density="7850">
+			<inertial density="13800">
 				<origin xyz="0.002084133424969194 -0.1180087385611795 0.10163798440735253" rpy="0 0 0"></origin>
 				<mass value="11.36414830883344"></mass>
@@ -13,5 +13,5 @@
 				</geometry>
 				<material name="">
-					<color rgba="1 1 1 1"></color>
+					<color rgba="1 0 0 1"></color>
 				</material>
 			</visual>

File: robotics/transbot-ros2ws/src/transbot_description/urdf/rigid_forklift/mobilebase/diff/diff.urdf.xacro (robot description, xacro)
@@ -13,5 +13,5 @@
 				</geometry>
 				<material name="">
-					<color rgba="1 1 1 1"></color>
+					<color rgba="1 1 0 1"></color>
 				</material>
 			</visual>

File: robotics/transbot-ros2ws/src/transbot_description/urdf/rigid_forklift/mobilebase/diff/wheel.urdf.xacro (robot description, xacro)
@@ -13,5 +13,5 @@
 				</geometry>
 				<material name="">
-					<color rgba="1 1 1 1"></color>
+					<color rgba="0.2 0.2 0.2 1"></color>
 				</material>
 			</visual>

File: robotics/transbot-ros2ws/src/transbot_description/urdf/rigid_forklift_wide/manipulator/horquilla.urdf.xacro (robot description, xacro)
@@ -13,5 +13,5 @@
 				</geometry>
 				<material name="">
-					<color rgba="1 1 1 1"></color>
+					<color rgba="0.2 0.7 0.2 1"></color>
 				</material>
 			</visual>

File: robotics/transbot-ros2ws/src/transbot_description/urdf/rigid_forklift_wide/manipulator/manipulator.urdf.xacro (robot description, xacro)
@@ -16,8 +16,8 @@
 			<child link="${prefix}${name}${suffix}horquilla"></child>
 			<axis xyz="0 0 1"></axis>
-			<limit lower="-0.05" upper="1.77" effort="1000000.0" velocity="1000000.0"></limit>
+			<limit lower="0.0" upper="1.27" effort="1000000.0" velocity="1000000.0"></limit>
 		</joint>
 		<joint name="j/${prefix}${name}${suffix}unna0" type="prismatic">
-			<origin xyz="0.075 -0.05 -0.05" rpy="0.0 0.0 0.0"></origin>
+			<origin xyz="0.075 -0.05 -0.1" rpy="0.0 0.0 0.0"></origin>
 			<parent link="${prefix}${name}${suffix}horquilla"></parent>
 			<child link="${prefix}${name}${suffix}unna0"></child>
@@ -26,5 +26,5 @@
 		</joint>
 		<joint name="j/${prefix}${name}${suffix}unna1" type="prismatic">
-			<origin xyz="0.075 0.05 -0.05" rpy="0.0 0.0 0.0"></origin>
+			<origin xyz="0.075 0.05 -0.1" rpy="0.0 0.0 0.0"></origin>
 			<parent link="${prefix}${name}${suffix}horquilla"></parent>
 			<child link="${prefix}${name}${suffix}unna1"></child>

File: robotics/transbot-ros2ws/src/transbot_description/urdf/rigid_forklift_wide/manipulator/portico.urdf.xacro (robot description, xacro)
@@ -4,7 +4,7 @@
 		<link name="${prefix}${name}${suffix}">
 			<inertial density="7850">
-				<origin xyz="6.334420083334617e-10 0.0 1.0591069298758413" rpy="0 0 0"></origin>
-				<mass value="1.914397192498048"></mass>
-				<inertia ixx="1.0821965894335586" ixy="-2.425319204727809e-10" ixz="1.2843361884440932e-09" iyy="0.7816162398331112" iyz="-9.934107462565105e-07" izz="0.30377101199216366"></inertia>
+				<origin xyz="6.16857676070328e-10 0.0 0.8229599125021437" rpy="0 0 0"></origin>
+				<mass value="1.4743995852768421"></mass>
+				<inertia ixx="0.5457702315565264" ixy="-1.2126596023639044e-10" ixz="7.484776801922124e-10" iyy="0.3235510188676326" iyz="2.483526865641276e-07" izz="0.22467654562206008"></inertia>
 			</inertial>
 			<visual>
@@ -13,5 +13,5 @@
 				</geometry>
 				<material name="">
-					<color rgba="1 1 1 1"></color>
+					<color rgba="0.7 0.2 0.2 1"></color>
 				</material>
 			</visual>

File: robotics/transbot-ros2ws/src/transbot_description/urdf/rigid_forklift_wide/manipulator/unna.urdf.xacro (robot description, xacro)
@@ -4,7 +4,7 @@
 		<link name="${prefix}${name}${suffix}">
 			<inertial density="7850">
-				<origin xyz="0.31713588379419205 -3.2682716149784016e-10 0.0016358343282475052" rpy="0 0 0"></origin>
-				<mass value="0.2319000195711851"></mass>
-				<inertia ixx="0.00014810430585443694" ixy="-2.4036117171074392e-11" ixz="0.0002657068439596089" iyy="0.011016142898947569" iyz="-1.2398188787661524e-13" izz="0.011085444903884207"></inertia>
+				<origin xyz="0.19335801902328506 3.8987254598624655e-10 0.01535802775643009" rpy="0 0 0"></origin>
+				<mass value="0.19440000566343466"></mass>
+				<inertia ixx="0.0003702513319354325" ixy="1.465484115391557e-11" ixz="0.0006457186385303325" iyy="0.005511267229784068" iyz="2.76272489497312e-12" izz="0.005323265933474595"></inertia>
 			</inertial>
 			<visual>
@@ -13,5 +13,5 @@
 				</geometry>
 				<material name="">
-					<color rgba="1 1 1 1"></color>
+					<color rgba="0.2 0.2 0.7 1"></color>
 				</material>
 			</visual>

File: robotics/transbot-ros2ws/src/transbot_description/urdf/rigid_forklift_wide/mobilebase/castor/arm.urdf.xacro (robot description, xacro)
@@ -4,7 +4,7 @@
 		<link name="${prefix}${name}${suffix}">
 			<inertial density="7850">
-				<origin xyz="0.023216223476559487 -5.499152560757377e-09 -0.023419604856066874" rpy="0 0 0"></origin>
+				<origin xyz="0.023216223476559487 -1.1854730520321233e-08 -0.023419604856066874" rpy="0 0 0"></origin>
 				<mass value="0.006568149425826657"></mass>
-				<inertia ixx="7.06487723744569e-06" ixy="-7.469593134069236e-13" ixz="1.2443357829905416e-06" iyy="4.505877976838242e-06" iyz="-2.7216179554656136e-12" izz="6.2024474186650775e-06"></inertia>
+				<inertia ixx="7.064875816359493e-06" ixy="-1.7161063013112547e-12" ixz="1.2443357829905416e-06" iyy="4.505877976838242e-06" iyz="-1.3739065952639405e-12" izz="6.202445997578881e-06"></inertia>
 			</inertial>
 			<visual>

File: robotics/transbot-ros2ws/src/transbot_description/urdf/rigid_forklift_wide/mobilebase/castor/wheel.urdf.xacro (robot description, xacro)
@@ -4,7 +4,7 @@
 		<link name="${prefix}${name}${suffix}">
 			<inertial density="2500">
-				<origin xyz="-1.4410434099052077e-09 -9.755815930202686e-11 -1.3427359559848857e-10" rpy="0 0 0"></origin>
+				<origin xyz="-1.4404439742105716e-09 -9.755815930202686e-11 -1.3427359559848857e-10" rpy="0 0 0"></origin>
 				<mass value="0.49389696990450227"></mass>
-				<inertia ixx="0.0005393656844413878" ixy="-1.6560826089644183e-12" ixz="-1.3026615866607103e-12" iyy="0.000539365805707347" iyz="1.1819249929968234e-13" izz="0.0009120414082038515"></inertia>
+				<inertia ixx="0.0005393656844413878" ixy="-1.6565452019202284e-12" ixz="-1.3026615867004634e-12" iyy="0.000539365805707347" iyz="1.1819249929968234e-13" izz="0.0009120414082038516"></inertia>
 			</inertial>
 			<visual>
@@ -13,5 +13,5 @@
 				</geometry>
 				<material name="">
-					<color rgba="1 1 1 1"></color>
+					<color rgba="0.2 0.2 0.2 1"></color>
 				</material>
 			</visual>

File: robotics/transbot-ros2ws/src/transbot_description/urdf/rigid_forklift_wide/mobilebase/chassis.urdf.xacro (robot description, xacro)
@@ -4,7 +4,7 @@
 		<link name="${prefix}${name}${suffix}">
 			<inertial density="7850">
-				<origin xyz="1.430045601294134e-07 0.0 0.12651649185789235" rpy="0 0 0"></origin>
-				<mass value="1.085422933101654"></mass>
-				<inertia ixx="0.11996343473625881" ixy="7.761021455128988e-09" ixz="3.515998706499306e-08" iyy="0.11004720866710413" iyz="-6.20881716410319e-08" izz="0.19016054769354823"></inertia>
+				<origin xyz="-2.034294682231643e-07 1.0171473411158215e-07 0.2282739023183229" rpy="0 0 0"></origin>
+				<mass value="2.2890552257498107"></mass>
+				<inertia ixx="0.2027274400644442" ixy="-7.761068819743012e-09" ixz="-1.0581325537136581e-07" iyy="0.1935426747453437" iyz="-8.939012034876226e-09" izz="0.3136757140357105"></inertia>
 			</inertial>
 			<visual>
@@ -13,5 +13,5 @@
 				</geometry>
 				<material name="">
-					<color rgba="1 1 1 1"></color>
+					<color rgba="1 1 0 1"></color>
 				</material>
 			</visual>

File: robotics/transbot-ros2ws/src/transbot_description/urdf/rigid_forklift_wide/mobilebase/control.urdf.xacro (robot description, xacro)
@@ -3,8 +3,8 @@
 	<xacro:macro name="control" params="prefix='' name='control' suffix=''">
 		<link name="${prefix}${name}${suffix}">
-			<inertial density="7850">
-				<origin xyz="-0.11800876511481027 0.09354560312818934 0.10163800234275462" rpy="0 0 0"></origin>
-				<mass value="11.364147067070007"></mass>
-				<inertia ixx="0.20224443786592244" ixy="0.04016673361813658" ixz="0.03380698382561664" iyy="0.1792783009602844" iyz="-0.02783002652166694" izz="0.2541928858214154"></inertia>
+			<inertial density="13800">
+				<origin xyz="0.002084133424969194 -0.1180087385611795 0.10163798440735253" rpy="0 0 0"></origin>
+				<mass value="11.36414830883344"></mass>
+				<inertia ixx="0.1792783214037889" ixy="-0.005400248580619397" ixz="0.0018980197654414812" iyy="0.17123017326450496" iyz="0.033806977088390505" izz="0.2231786465435561"></inertia>
 			</inertial>
 			<visual>
@@ -13,5 +13,5 @@
 				</geometry>
 				<material name="">
-					<color rgba="1 1 1 1"></color>
+					<color rgba="1 0 0 1"></color>
 				</material>
 			</visual>

File: robotics/transbot-ros2ws/src/transbot_description/urdf/rigid_forklift_wide/mobilebase/diff/diff.urdf.xacro (robot description, xacro)
@@ -13,5 +13,5 @@
 				</geometry>
 				<material name="">
-					<color rgba="1 1 1 1"></color>
+					<color rgba="1 1 0 1"></color>
 				</material>
 			</visual>

File: robotics/transbot-ros2ws/src/transbot_description/urdf/rigid_forklift_wide/mobilebase/diff/wheel.urdf.xacro (robot description, xacro)
@@ -13,5 +13,5 @@
 				</geometry>
 				<material name="">
-					<color rgba="1 1 1 1"></color>
+					<color rgba="0.2 0.2 0.2 1"></color>
 				</material>
 			</visual>

File: robotics/transbot-ros2ws/src/transbot_description/urdf/rigid_forklift_wide/mobilebase/mobilebase.urdf.xacro (robot description, xacro)
@@ -28,8 +28,9 @@
 		</joint>
 		<joint name="j/${prefix}${name}${suffix}control" type="prismatic">
-			<origin xyz="0.0 0.0 0.17" rpy="0.0 0.0 0.0"></origin>
+			<origin xyz="0.075 0.0 0.17" rpy="0.0 0.0 1.5707963267948966"></origin>
 			<parent link="${prefix}${name}${suffix}_"></parent>
 			<child link="${prefix}${name}${suffix}control"></child>
-			<axis xyz="1 0 0"></axis>
+			<dynamics damping="10" friction="10"></dynamics>
+			<axis xyz="0 -1 0"></axis>
 			<limit lower="0.0" upper="0.5" effort="1000000.0" velocity="1000000.0"></limit>
 		</joint>

File: robotics/transbot-ros2ws/src/transbot_description/urdf/robot_arm/arm/link0.urdf.xacro (robot description, xacro)
@@ -4,7 +4,7 @@
 		<link name="${prefix}${name}${suffix}">
 			<inertial density="7850">
-				<origin xyz="-1.9585539810652476e-10 2.49600873563491e-10 0.0775319300078531" rpy="0 0 0"></origin>
+				<origin xyz="3.264256635108746e-10 7.718819351808904e-10 0.0775319300078531" rpy="0 0 0"></origin>
 				<mass value="1.16092626315852"></mass>
-				<inertia ixx="0.010230603676813953" ixy="-6.347515111798829e-11" ixz="-2.5837893971342154e-11" iyy="0.010230602464154349" iyz="-4.729087447709836e-11" izz="0.005150119492706533"></inertia>
+				<inertia ixx="0.010230603676813953" ixy="-6.347515076872623e-11" ixz="2.1172025735572452e-11" iyy="0.010230602464154349" iyz="-5.96529665626454e-12" izz="0.005150119492706532"></inertia>
 			</inertial>
 			<visual>
@@ -13,5 +13,5 @@
 				</geometry>
 				<material name="">
-					<color rgba="1 1 1 1"></color>
+					<color rgba="1 0 0 1"></color>
 				</material>
 			</visual>
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