Commit message: added odometry to gazebo exports

File: robotics/transbot-ros2ws/src/transbot_description/urdf/rigid_forklift_wide/manipulator/horquilla.urdf.xacro (robot description, xacro)
@@ -10,5 +10,5 @@
 			<visual>
 				<geometry>
-					<mesh filename="file:$(find transbot_description)/meshes/rigid_forklift_wide/manipulator/horquilla.stl" scale="1e-3 1e-3 1e-3"></mesh>
+					<mesh filename="package://transbot_description/meshes/rigid_forklift_wide/manipulator/horquilla.stl" scale="1e-3 1e-3 1e-3"></mesh>
 				</geometry>
 				<material name="">
@@ -18,5 +18,5 @@
 			<collision>
 				<geometry>
-					<mesh filename="file:$(find transbot_description)/meshes/rigid_forklift_wide/manipulator/horquilla.stl" scale="1e-3 1e-3 1e-3"></mesh>
+					<mesh filename="package://transbot_description/meshes/rigid_forklift_wide/manipulator/horquilla.stl" scale="1e-3 1e-3 1e-3"></mesh>
 				</geometry>
 			</collision>

File: robotics/transbot-ros2ws/src/transbot_description/urdf/rigid_forklift_wide/manipulator/manipulator.urdf.xacro (robot description, xacro)
@@ -23,5 +23,5 @@
 			<child link="${prefix}${name}${suffix}unna0"></child>
 			<axis xyz="0 -1 0"></axis>
-			<limit lower="0.325" upper="0.0" effort="1000000.0" velocity="1000000.0"></limit>
+			<limit lower="0.0" upper="0.325" effort="1000000.0" velocity="1000000.0"></limit>
 		</joint>
 		<joint name="j/${prefix}${name}${suffix}unna1" type="prismatic">
@@ -31,5 +31,5 @@
 			<mimic joint="j/${prefix}${name}${suffix}unna0" multiplier="1" offset="0"></mimic>
 			<axis xyz="0 1 0"></axis>
-			<limit lower="0.325" upper="0.0" effort="1000000.0" velocity="1000000.0"></limit>
+			<limit lower="0.0" upper="0.325" effort="1000000.0" velocity="1000000.0"></limit>
 		</joint>
 		<xacro:portico prefix="${prefix}${name}${suffix}" suffix=""></xacro:portico>

File: robotics/transbot-ros2ws/src/transbot_description/urdf/rigid_forklift_wide/manipulator/portico.urdf.xacro (robot description, xacro)
@@ -10,5 +10,5 @@
 			<visual>
 				<geometry>
-					<mesh filename="file:$(find transbot_description)/meshes/rigid_forklift_wide/manipulator/portico.stl" scale="1e-3 1e-3 1e-3"></mesh>
+					<mesh filename="package://transbot_description/meshes/rigid_forklift_wide/manipulator/portico.stl" scale="1e-3 1e-3 1e-3"></mesh>
 				</geometry>
 				<material name="">
@@ -18,5 +18,5 @@
 			<collision>
 				<geometry>
-					<mesh filename="file:$(find transbot_description)/meshes/rigid_forklift_wide/manipulator/portico.stl" scale="1e-3 1e-3 1e-3"></mesh>
+					<mesh filename="package://transbot_description/meshes/rigid_forklift_wide/manipulator/portico.stl" scale="1e-3 1e-3 1e-3"></mesh>
 				</geometry>
 			</collision>

File: robotics/transbot-ros2ws/src/transbot_description/urdf/rigid_forklift_wide/manipulator/unna.urdf.xacro (robot description, xacro)
@@ -10,5 +10,5 @@
 			<visual>
 				<geometry>
-					<mesh filename="file:$(find transbot_description)/meshes/rigid_forklift_wide/manipulator/unna.stl" scale="1e-3 1e-3 1e-3"></mesh>
+					<mesh filename="package://transbot_description/meshes/rigid_forklift_wide/manipulator/unna.stl" scale="1e-3 1e-3 1e-3"></mesh>
 				</geometry>
 				<material name="">
@@ -18,5 +18,5 @@
 			<collision>
 				<geometry>
-					<mesh filename="file:$(find transbot_description)/meshes/rigid_forklift_wide/manipulator/unna.stl" scale="1e-3 1e-3 1e-3"></mesh>
+					<mesh filename="package://transbot_description/meshes/rigid_forklift_wide/manipulator/unna.stl" scale="1e-3 1e-3 1e-3"></mesh>
 				</geometry>
 			</collision>

File: robotics/transbot-ros2ws/src/transbot_description/urdf/rigid_forklift_wide/mobilebase/castor/arm.urdf.xacro (robot description, xacro)
@@ -10,5 +10,5 @@
 			<visual>
 				<geometry>
-					<mesh filename="file:$(find transbot_description)/meshes/rigid_forklift_wide/mobilebase/castor/arm.stl" scale="1e-3 1e-3 1e-3"></mesh>
+					<mesh filename="package://transbot_description/meshes/rigid_forklift_wide/mobilebase/castor/arm.stl" scale="1e-3 1e-3 1e-3"></mesh>
 				</geometry>
 				<material name="">
@@ -18,5 +18,5 @@
 			<collision>
 				<geometry>
-					<mesh filename="file:$(find transbot_description)/meshes/rigid_forklift_wide/mobilebase/castor/arm.stl" scale="1e-3 1e-3 1e-3"></mesh>
+					<mesh filename="package://transbot_description/meshes/rigid_forklift_wide/mobilebase/castor/arm.stl" scale="1e-3 1e-3 1e-3"></mesh>
 				</geometry>
 			</collision>

File: robotics/transbot-ros2ws/src/transbot_description/urdf/rigid_forklift_wide/mobilebase/castor/castor.urdf.xacro (robot description, xacro)
@@ -10,5 +10,5 @@
 			<visual>
 				<geometry>
-					<mesh filename="file:$(find transbot_description)/meshes/rigid_forklift_wide/mobilebase/castor/_.stl" scale="1e-3 1e-3 1e-3"></mesh>
+					<mesh filename="package://transbot_description/meshes/rigid_forklift_wide/mobilebase/castor/_.stl" scale="1e-3 1e-3 1e-3"></mesh>
 				</geometry>
 				<material name="">
@@ -18,5 +18,5 @@
 			<collision>
 				<geometry>
-					<mesh filename="file:$(find transbot_description)/meshes/rigid_forklift_wide/mobilebase/castor/_.stl" scale="1e-3 1e-3 1e-3"></mesh>
+					<mesh filename="package://transbot_description/meshes/rigid_forklift_wide/mobilebase/castor/_.stl" scale="1e-3 1e-3 1e-3"></mesh>
 				</geometry>
 			</collision>

File: robotics/transbot-ros2ws/src/transbot_description/urdf/rigid_forklift_wide/mobilebase/castor/wheel.urdf.xacro (robot description, xacro)
@@ -4,11 +4,11 @@
 		<link name="${prefix}${name}${suffix}">
 			<inertial density="2500">
-				<origin xyz="-1.4404439742105716e-09 -9.755815930202686e-11 -1.3427359559848857e-10" rpy="0 0 0"></origin>
+				<origin xyz="-7.130287587696525e-10 -2.809854818606764e-10 -1.3427359559848857e-10" rpy="0 0 0"></origin>
 				<mass value="0.49389696990450227"></mass>
-				<inertia ixx="0.0005393656844413878" ixy="-1.6565452019202284e-12" ixz="-1.3026615867004634e-12" iyy="0.000539365805707347" iyz="1.1819249929968234e-13" izz="0.0009120414082038516"></inertia>
+				<inertia ixx="0.0005393656238084077" ixy="-7.086922650997735e-13" ixz="-1.3026616349406924e-12" iyy="0.0005393657450743677" iyz="1.1819251146409114e-13" izz="0.0009120412869378921"></inertia>
 			</inertial>
 			<visual>
 				<geometry>
-					<mesh filename="file:$(find transbot_description)/meshes/rigid_forklift_wide/mobilebase/castor/wheel.stl" scale="1e-3 1e-3 1e-3"></mesh>
+					<mesh filename="package://transbot_description/meshes/rigid_forklift_wide/mobilebase/castor/wheel.stl" scale="1e-3 1e-3 1e-3"></mesh>
 				</geometry>
 				<material name="">
@@ -18,5 +18,5 @@
 			<collision>
 				<geometry>
-					<mesh filename="file:$(find transbot_description)/meshes/rigid_forklift_wide/mobilebase/castor/wheel.stl" scale="1e-3 1e-3 1e-3"></mesh>
+					<mesh filename="package://transbot_description/meshes/rigid_forklift_wide/mobilebase/castor/wheel.stl" scale="1e-3 1e-3 1e-3"></mesh>
 				</geometry>
 			</collision>

File: robotics/transbot-ros2ws/src/transbot_description/urdf/rigid_forklift_wide/mobilebase/chassis.urdf.xacro (robot description, xacro)
@@ -10,5 +10,5 @@
 			<visual>
 				<geometry>
-					<mesh filename="file:$(find transbot_description)/meshes/rigid_forklift_wide/mobilebase/chassis.stl" scale="1e-3 1e-3 1e-3"></mesh>
+					<mesh filename="package://transbot_description/meshes/rigid_forklift_wide/mobilebase/chassis.stl" scale="1e-3 1e-3 1e-3"></mesh>
 				</geometry>
 				<material name="">
@@ -18,5 +18,5 @@
 			<collision>
 				<geometry>
-					<mesh filename="file:$(find transbot_description)/meshes/rigid_forklift_wide/mobilebase/chassis.stl" scale="1e-3 1e-3 1e-3"></mesh>
+					<mesh filename="package://transbot_description/meshes/rigid_forklift_wide/mobilebase/chassis.stl" scale="1e-3 1e-3 1e-3"></mesh>
 				</geometry>
 			</collision>

File: robotics/transbot-ros2ws/src/transbot_description/urdf/rigid_forklift_wide/mobilebase/control.urdf.xacro (robot description, xacro)
@@ -4,11 +4,11 @@
 		<link name="${prefix}${name}${suffix}">
 			<inertial density="13800">
-				<origin xyz="0.002084133424969194 -0.1180087385611795 0.10163798440735253" rpy="0 0 0"></origin>
-				<mass value="11.36414830883344"></mass>
-				<inertia ixx="0.1792783214037889" ixy="-0.005400248580619397" ixz="0.0018980197654414812" iyy="0.17123017326450496" iyz="0.033806977088390505" izz="0.2231786465435561"></inertia>
+				<origin xyz="0.006921931017760558 -0.04374911256185983 0.016953211369279058" rpy="0 0 0"></origin>
+				<mass value="3.4216465428471565"></mass>
+				<inertia ixx="0.06684930260049168" ixy="-0.0036414557355901483" ixz="-0.00010768790123973424" iyy="0.07845860219646296" iyz="0.0030195033418340465" izz="0.14366063335138574"></inertia>
 			</inertial>
 			<visual>
 				<geometry>
-					<mesh filename="file:$(find transbot_description)/meshes/rigid_forklift_wide/mobilebase/control.stl" scale="1e-3 1e-3 1e-3"></mesh>
+					<mesh filename="package://transbot_description/meshes/rigid_forklift_wide/mobilebase/control.stl" scale="1e-3 1e-3 1e-3"></mesh>
 				</geometry>
 				<material name="">
@@ -18,5 +18,5 @@
 			<collision>
 				<geometry>
-					<mesh filename="file:$(find transbot_description)/meshes/rigid_forklift_wide/mobilebase/control.stl" scale="1e-3 1e-3 1e-3"></mesh>
+					<mesh filename="package://transbot_description/meshes/rigid_forklift_wide/mobilebase/control.stl" scale="1e-3 1e-3 1e-3"></mesh>
 				</geometry>
 			</collision>

File: robotics/transbot-ros2ws/src/transbot_description/urdf/rigid_forklift_wide/mobilebase/diff/diff.urdf.xacro (robot description, xacro)
@@ -10,5 +10,5 @@
 			<visual>
 				<geometry>
-					<mesh filename="file:$(find transbot_description)/meshes/rigid_forklift_wide/mobilebase/diff/_.stl" scale="1e-3 1e-3 1e-3"></mesh>
+					<mesh filename="package://transbot_description/meshes/rigid_forklift_wide/mobilebase/diff/_.stl" scale="1e-3 1e-3 1e-3"></mesh>
 				</geometry>
 				<material name="">
@@ -18,5 +18,5 @@
 			<collision>
 				<geometry>
-					<mesh filename="file:$(find transbot_description)/meshes/rigid_forklift_wide/mobilebase/diff/_.stl" scale="1e-3 1e-3 1e-3"></mesh>
+					<mesh filename="package://transbot_description/meshes/rigid_forklift_wide/mobilebase/diff/_.stl" scale="1e-3 1e-3 1e-3"></mesh>
 				</geometry>
 			</collision>

File: robotics/transbot-ros2ws/src/transbot_description/urdf/rigid_forklift_wide/mobilebase/diff/wheel.urdf.xacro (robot description, xacro)
@@ -4,11 +4,11 @@
 		<link name="${prefix}${name}${suffix}">
 			<inertial density="2500">
-				<origin xyz="1.1788708620254621e-09 5.703497958218067e-10 -2.1101991334018597e-10" rpy="0 0 0"></origin>
+				<origin xyz="1.1795472079015525e-09 5.700142648598401e-10 -2.1101991334018597e-10" rpy="0 0 0"></origin>
 				<mass value="0.43773383367806673"></mass>
-				<inertia ixx="0.00046364856795359305" ixy="-6.391183584106932e-12" ixz="-3.5527147677300667e-13" iyy="0.0004636485376371025" iyz="-5.268352755424735e-20" izz="0.0008105681445158545"></inertia>
+				<inertia ixx="0.00046364856795359305" ixy="-6.390171662083665e-12" ixz="-3.552714768354811e-13" iyy="0.0004636485376371025" iyz="4.625402743927758e-16" izz="0.0008105681445158545"></inertia>
 			</inertial>
 			<visual>
 				<geometry>
-					<mesh filename="file:$(find transbot_description)/meshes/rigid_forklift_wide/mobilebase/diff/wheel.stl" scale="1e-3 1e-3 1e-3"></mesh>
+					<mesh filename="package://transbot_description/meshes/rigid_forklift_wide/mobilebase/diff/wheel.stl" scale="1e-3 1e-3 1e-3"></mesh>
 				</geometry>
 				<material name="">
@@ -18,5 +18,5 @@
 			<collision>
 				<geometry>
-					<mesh filename="file:$(find transbot_description)/meshes/rigid_forklift_wide/mobilebase/diff/wheel.stl" scale="1e-3 1e-3 1e-3"></mesh>
+					<mesh filename="package://transbot_description/meshes/rigid_forklift_wide/mobilebase/diff/wheel.stl" scale="1e-3 1e-3 1e-3"></mesh>
 				</geometry>
 			</collision>

File: robotics/transbot-ros2ws/src/transbot_gazebo/urdf/rigid_forklift_wide/__all__.urdf.xacro (robot description, xacro)
@@ -1,14 +1,32 @@
 <?xml version="1.0" encoding="utf-8"?>
 <robot xmlns:xacro="http://www.ros.org/wiki/xacro" name="rigid_forklift_wide">
+	<xacro:arg name="robot_name" default="transbot"></xacro:arg>
 	<xacro:arg name="ros2_control_namespace" default="/transbot"></xacro:arg>
-	<xacro:arg name="ros2_control_dict" default="rigid_forklift_wide//ros2_control.yaml"></xacro:arg>
+	<xacro:arg name="ros2_control_dict" default="rigid_forklift_wide.yaml"></xacro:arg>
+	<xacro:arg name="ros2_control_pkg" default="transbot_controller"></xacro:arg>
+	<xacro:arg name="gz_odometry_frame_prefix" default=""></xacro:arg>
+	<xacro:arg name="gz_odometry_frame" default="odom"></xacro:arg>
+	<xacro:property name="_ros2_control_pkg" value="$(arg ros2_control_pkg)"></xacro:property>
+	<xacro:property name="_ros2_control_path" value="$(find ${_ros2_control_pkg})"></xacro:property>
 	<xacro:include filename="$(find transbot_description)/urdf/rigid_forklift_wide/__all__.urdf.xacro"></xacro:include>
 	<xacro:include filename="$(find transbot_gazebo)/urdf/rigid_forklift_wide/rigid_forklift_wide.urdf.xacro"></xacro:include>
+	<xacro:include filename="$(find transbot_gazebo)/urdf/rigid_forklift_wide/__extras__.urdf.xacro"></xacro:include>
 	<gazebo>
 		<plugin filename="gz_ros2_control-system" name="gz_ros2_control::GazeboSimROS2ControlPlugin">
-			<parameters>$(find transbot_gazebo)/config/$(arg ros2_control_dict)</parameters>
+			<parameters>${_ros2_control_path}/config/$(arg ros2_control_dict)</parameters>
 			<ros>
 				<namespace>$(arg ros2_control_namespace)</namespace>
 			</ros>
+		</plugin>
+	</gazebo>
+	<gazebo>
+		<plugin filename="gz-sim-odometry-publisher-system" name="gz::sim::systems::OdometryPublisher">
+			<odom_frame>$(arg gz_odometry_frame_prefix)/$(arg gz_odometry_frame)</odom_frame>
+			<robot_base_frame>$(arg gz_odometry_frame_prefix)/gz_gtruth</robot_base_frame>
+			<odom_topic>/model/$(arg robot_name)/ground_truth/odometry</odom_topic>
+			<tf_topic>/model/$(arg robot_name)/ground_truth/pose</tf_topic>
+			<odom_publish_rate>50</odom_publish_rate>
+			<dimensions>3</dimensions>
+			<gaussian_noise>0.0</gaussian_noise>
 		</plugin>
 	</gazebo>

File: robotics/transbot-ros2ws/src/transbot_gazebo/urdf/rigid_forklift_wide/manipulator/__all__.urdf.xacro (robot description, xacro)
@@ -1,14 +1,32 @@
 <?xml version="1.0" encoding="utf-8"?>
 <robot xmlns:xacro="http://www.ros.org/wiki/xacro" name="manipulator">
+	<xacro:arg name="robot_name" default="transbot"></xacro:arg>
 	<xacro:arg name="ros2_control_namespace" default="/transbot"></xacro:arg>
-	<xacro:arg name="ros2_control_dict" default="rigid_forklift_wide//ros2_control.yaml"></xacro:arg>
+	<xacro:arg name="ros2_control_dict" default="rigid_forklift_wide.yaml"></xacro:arg>
+	<xacro:arg name="ros2_control_pkg" default="transbot_controller"></xacro:arg>
+	<xacro:arg name="gz_odometry_frame_prefix" default=""></xacro:arg>
+	<xacro:arg name="gz_odometry_frame" default="odom"></xacro:arg>
+	<xacro:property name="_ros2_control_pkg" value="$(arg ros2_control_pkg)"></xacro:property>
+	<xacro:property name="_ros2_control_path" value="$(find ${_ros2_control_pkg})"></xacro:property>
 	<xacro:include filename="$(find transbot_description)/urdf/rigid_forklift_wide/__all__.urdf.xacro"></xacro:include>
 	<xacro:include filename="$(find transbot_gazebo)/urdf/rigid_forklift_wide/manipulator.urdf.xacro"></xacro:include>
+	<xacro:include filename="$(find transbot_gazebo)/urdf/rigid_forklift_wide/__extras__.urdf.xacro"></xacro:include>
 	<gazebo>
 		<plugin filename="gz_ros2_control-system" name="gz_ros2_control::GazeboSimROS2ControlPlugin">
-			<parameters>$(find transbot_gazebo)/config/$(arg ros2_control_dict)</parameters>
+			<parameters>${_ros2_control_path}/config/$(arg ros2_control_dict)</parameters>
 			<ros>
 				<namespace>$(arg ros2_control_namespace)</namespace>
 			</ros>
+		</plugin>
+	</gazebo>
+	<gazebo>
+		<plugin filename="gz-sim-odometry-publisher-system" name="gz::sim::systems::OdometryPublisher">
+			<odom_frame>$(arg gz_odometry_frame_prefix)/$(arg gz_odometry_frame)</odom_frame>
+			<robot_base_frame>$(arg gz_odometry_frame_prefix)/gz_gtruth</robot_base_frame>
+			<odom_topic>/model/$(arg robot_name)/ground_truth/odometry</odom_topic>
+			<tf_topic>/model/$(arg robot_name)/ground_truth/pose</tf_topic>
+			<odom_publish_rate>50</odom_publish_rate>
+			<dimensions>3</dimensions>
+			<gaussian_noise>0.0</gaussian_noise>
 		</plugin>
 	</gazebo>

File: robotics/transbot-ros2ws/src/transbot_gazebo/urdf/rigid_forklift_wide/mobilebase/__all__.urdf.xacro (robot description, xacro)
@@ -1,14 +1,32 @@
 <?xml version="1.0" encoding="utf-8"?>
 <robot xmlns:xacro="http://www.ros.org/wiki/xacro" name="mobilebase">
+	<xacro:arg name="robot_name" default="transbot"></xacro:arg>
 	<xacro:arg name="ros2_control_namespace" default="/transbot"></xacro:arg>
-	<xacro:arg name="ros2_control_dict" default="rigid_forklift_wide//ros2_control.yaml"></xacro:arg>
+	<xacro:arg name="ros2_control_dict" default="rigid_forklift_wide.yaml"></xacro:arg>
+	<xacro:arg name="ros2_control_pkg" default="transbot_controller"></xacro:arg>
+	<xacro:arg name="gz_odometry_frame_prefix" default=""></xacro:arg>
+	<xacro:arg name="gz_odometry_frame" default="odom"></xacro:arg>
+	<xacro:property name="_ros2_control_pkg" value="$(arg ros2_control_pkg)"></xacro:property>
+	<xacro:property name="_ros2_control_path" value="$(find ${_ros2_control_pkg})"></xacro:property>
 	<xacro:include filename="$(find transbot_description)/urdf/rigid_forklift_wide/__all__.urdf.xacro"></xacro:include>
 	<xacro:include filename="$(find transbot_gazebo)/urdf/rigid_forklift_wide/mobilebase.urdf.xacro"></xacro:include>
+	<xacro:include filename="$(find transbot_gazebo)/urdf/rigid_forklift_wide/__extras__.urdf.xacro"></xacro:include>
 	<gazebo>
 		<plugin filename="gz_ros2_control-system" name="gz_ros2_control::GazeboSimROS2ControlPlugin">
-			<parameters>$(find transbot_gazebo)/config/$(arg ros2_control_dict)</parameters>
+			<parameters>${_ros2_control_path}/config/$(arg ros2_control_dict)</parameters>
 			<ros>
 				<namespace>$(arg ros2_control_namespace)</namespace>
 			</ros>
+		</plugin>
+	</gazebo>
+	<gazebo>
+		<plugin filename="gz-sim-odometry-publisher-system" name="gz::sim::systems::OdometryPublisher">
+			<odom_frame>$(arg gz_odometry_frame_prefix)/$(arg gz_odometry_frame)</odom_frame>
+			<robot_base_frame>$(arg gz_odometry_frame_prefix)/gz_gtruth</robot_base_frame>
+			<odom_topic>/model/$(arg robot_name)/ground_truth/odometry</odom_topic>
+			<tf_topic>/model/$(arg robot_name)/ground_truth/pose</tf_topic>
+			<odom_publish_rate>50</odom_publish_rate>
+			<dimensions>3</dimensions>
+			<gaussian_noise>0.0</gaussian_noise>
 		</plugin>
 	</gazebo>

File: robotics/transbot-ros2ws/src/transbot_gazebo/urdf/rigid_forklift_wide/mobilebase/castor/__all__.urdf.xacro (robot description, xacro)
@@ -1,14 +1,32 @@
 <?xml version="1.0" encoding="utf-8"?>
 <robot xmlns:xacro="http://www.ros.org/wiki/xacro" name="castor">
+	<xacro:arg name="robot_name" default="transbot"></xacro:arg>
 	<xacro:arg name="ros2_control_namespace" default="/transbot"></xacro:arg>
-	<xacro:arg name="ros2_control_dict" default="rigid_forklift_wide/mobilebase/ros2_control.yaml"></xacro:arg>
+	<xacro:arg name="ros2_control_dict" default="rigid_forklift_wide/mobilebase.yaml"></xacro:arg>
+	<xacro:arg name="ros2_control_pkg" default="transbot_controller"></xacro:arg>
+	<xacro:arg name="gz_odometry_frame_prefix" default=""></xacro:arg>
+	<xacro:arg name="gz_odometry_frame" default="odom"></xacro:arg>
+	<xacro:property name="_ros2_control_pkg" value="$(arg ros2_control_pkg)"></xacro:property>
+	<xacro:property name="_ros2_control_path" value="$(find ${_ros2_control_pkg})"></xacro:property>
 	<xacro:include filename="$(find transbot_description)/urdf/rigid_forklift_wide/mobilebase/__all__.urdf.xacro"></xacro:include>
 	<xacro:include filename="$(find transbot_gazebo)/urdf/rigid_forklift_wide/mobilebase/castor.urdf.xacro"></xacro:include>
+	<xacro:include filename="$(find transbot_gazebo)/urdf/rigid_forklift_wide/mobilebase/__extras__.urdf.xacro"></xacro:include>
 	<gazebo>
 		<plugin filename="gz_ros2_control-system" name="gz_ros2_control::GazeboSimROS2ControlPlugin">
-			<parameters>$(find transbot_gazebo)/config/$(arg ros2_control_dict)</parameters>
+			<parameters>${_ros2_control_path}/config/$(arg ros2_control_dict)</parameters>
 			<ros>
 				<namespace>$(arg ros2_control_namespace)</namespace>
 			</ros>
+		</plugin>
+	</gazebo>
+	<gazebo>
+		<plugin filename="gz-sim-odometry-publisher-system" name="gz::sim::systems::OdometryPublisher">
+			<odom_frame>$(arg gz_odometry_frame_prefix)/$(arg gz_odometry_frame)</odom_frame>
+			<robot_base_frame>$(arg gz_odometry_frame_prefix)/gz_gtruth</robot_base_frame>
+			<odom_topic>/model/$(arg robot_name)/ground_truth/odometry</odom_topic>
+			<tf_topic>/model/$(arg robot_name)/ground_truth/pose</tf_topic>
+			<odom_publish_rate>50</odom_publish_rate>
+			<dimensions>3</dimensions>
+			<gaussian_noise>0.0</gaussian_noise>
 		</plugin>
 	</gazebo>
