Commit message: rounded wheels

File: robotics/transbot-ros2ws/src/transbot_description/urdf/shelf_lifter/mobilebase/castor/arm.urdf.xacro (robot description, xacro)
@@ -4,7 +4,7 @@
 		<link name="${prefix}${name}${suffix}">
 			<inertial density="7850">
-				<origin xyz="0.023216224918960162 -5.499152560757377e-09 -0.023419614952871575" rpy="0 0 0"></origin>
+				<origin xyz="0.023216223476559487 -5.499152560757377e-09 -0.023419604856066874" rpy="0 0 0"></origin>
 				<mass value="0.006568149425826657"></mass>
-				<inertia ixx="7.064874131194068e-06" ixy="-7.441838079437996e-13" ixz="1.2443340214776094e-06" iyy="4.505874430690099e-06" iyz="-2.7216175907765425e-12" izz="6.202446978768557e-06"></inertia>
+				<inertia ixx="7.06487723744569e-06" ixy="-7.469593134069236e-13" ixz="1.2443357829905416e-06" iyy="4.505877976838242e-06" iyz="-2.7216179554656136e-12" izz="6.2024474186650775e-06"></inertia>
 			</inertial>
 			<visual>

File: robotics/transbot-ros2ws/src/transbot_description/urdf/shelf_lifter/mobilebase/castor/wheel.urdf.xacro (robot description, xacro)
@@ -4,7 +4,7 @@
 		<link name="${prefix}${name}${suffix}">
 			<inertial density="2500">
-				<origin xyz="-7.118298873803803e-10 -2.809854818606764e-10 -1.3427359559848857e-10" rpy="0 0 0"></origin>
-				<mass value="0.49389696990450227"></mass>
-				<inertia ixx="0.0005393656238084077" ixy="-7.086922652661503e-13" ixz="-1.3026616350201983e-12" iyy="0.0005393657450743677" iyz="1.1819251146409114e-13" izz="0.0009120412869378921"></inertia>
+				<origin xyz="1.4340148303551888e-09 -3.5090750499906038e-09 -2.852402266199148e-10" rpy="0 0 0"></origin>
+				<mass value="0.4594138978670041"></mass>
+				<inertia ixx="0.00047094974130837766" ixy="-1.5209132563311692e-11" ixz="1.9058826710217818e-12" iyy="0.00047094934719401157" iyz="-1.2603575130752765e-11" izz="0.0008008167848553598"></inertia>
 			</inertial>
 			<visual>

File: robotics/transbot-ros2ws/src/transbot_description/urdf/shelf_lifter/mobilebase/doublebar/diff/wheel.urdf.xacro (robot description, xacro)
@@ -4,7 +4,7 @@
 		<link name="${prefix}${name}${suffix}">
 			<inertial density="2500">
-				<origin xyz="1.0145187241984178e-11 -3.3865903162148433e-10 -2.110198946332709e-10" rpy="0 0 0"></origin>
-				<mass value="0.437733872483174"></mass>
-				<inertia ixx="0.00046364856795359316" ixy="-4.0227080940624326e-12" ixz="-3.5527136881716666e-13" iyy="0.0004636485679535932" iyz="3.128212292636545e-20" izz="0.0008105681748323452"></inertia>
+				<origin xyz="4.752325537276356e-09 -4.403267049900442e-10 1.1552381330584986e-09" rpy="0 0 0"></origin>
+				<mass value="0.40324983031799394"></mass>
+				<inertia ixx="0.00039830266587159653" ixy="1.0545151870168692e-11" ixz="7.179444439778207e-12" iyy="0.0003983027871375477" iyz="-7.221077640592899e-13" izz="0.0006993444306620614"></inertia>
 			</inertial>
 			<visual>

File: robotics/transbot-ros2ws/src/transbot_gazebo/urdf/shelf_lifter/__all__.urdf.xacro (robot description, xacro)
@@ -1,14 +1,32 @@
 <?xml version="1.0" encoding="utf-8"?>
 <robot xmlns:xacro="http://www.ros.org/wiki/xacro" name="shelf_lifter">
+	<xacro:arg name="robot_name" default="transbot"></xacro:arg>
 	<xacro:arg name="ros2_control_namespace" default="/transbot"></xacro:arg>
-	<xacro:arg name="ros2_control_dict" default="shelf_lifter//ros2_control.yaml"></xacro:arg>
+	<xacro:arg name="ros2_control_dict" default="shelf_lifter.yaml"></xacro:arg>
+	<xacro:arg name="ros2_control_pkg" default="transbot_controller"></xacro:arg>
+	<xacro:arg name="gz_odometry_frame_prefix" default=""></xacro:arg>
+	<xacro:arg name="gz_odometry_frame" default="odom"></xacro:arg>
+	<xacro:property name="_ros2_control_pkg" value="$(arg ros2_control_pkg)"></xacro:property>
+	<xacro:property name="_ros2_control_path" value="$(find ${_ros2_control_pkg})"></xacro:property>
 	<xacro:include filename="$(find transbot_description)/urdf/shelf_lifter/__all__.urdf.xacro"></xacro:include>
 	<xacro:include filename="$(find transbot_gazebo)/urdf/shelf_lifter/shelf_lifter.urdf.xacro"></xacro:include>
+	<xacro:include filename="$(find transbot_gazebo)/urdf/shelf_lifter/__extras__.urdf.xacro"></xacro:include>
 	<gazebo>
 		<plugin filename="gz_ros2_control-system" name="gz_ros2_control::GazeboSimROS2ControlPlugin">
-			<parameters>$(find transbot_gazebo)/config/$(arg ros2_control_dict)</parameters>
+			<parameters>${_ros2_control_path}/config/$(arg ros2_control_dict)</parameters>
 			<ros>
 				<namespace>$(arg ros2_control_namespace)</namespace>
 			</ros>
+		</plugin>
+	</gazebo>
+	<gazebo>
+		<plugin filename="gz-sim-odometry-publisher-system" name="gz::sim::systems::OdometryPublisher">
+			<odom_frame>$(arg gz_odometry_frame_prefix)/$(arg gz_odometry_frame)</odom_frame>
+			<robot_base_frame>$(arg gz_odometry_frame_prefix)/gz_gtruth</robot_base_frame>
+			<odom_topic>/model/$(arg robot_name)/ground_truth/odometry</odom_topic>
+			<tf_topic>/model/$(arg robot_name)/ground_truth/pose</tf_topic>
+			<odom_publish_rate>50</odom_publish_rate>
+			<dimensions>3</dimensions>
+			<gaussian_noise>0.0</gaussian_noise>
 		</plugin>
 	</gazebo>

File: robotics/transbot-ros2ws/src/transbot_gazebo/urdf/shelf_lifter/mobilebase/__all__.urdf.xacro (robot description, xacro)
@@ -1,14 +1,32 @@
 <?xml version="1.0" encoding="utf-8"?>
 <robot xmlns:xacro="http://www.ros.org/wiki/xacro" name="mobilebase">
+	<xacro:arg name="robot_name" default="transbot"></xacro:arg>
 	<xacro:arg name="ros2_control_namespace" default="/transbot"></xacro:arg>
-	<xacro:arg name="ros2_control_dict" default="shelf_lifter//ros2_control.yaml"></xacro:arg>
+	<xacro:arg name="ros2_control_dict" default="shelf_lifter.yaml"></xacro:arg>
+	<xacro:arg name="ros2_control_pkg" default="transbot_controller"></xacro:arg>
+	<xacro:arg name="gz_odometry_frame_prefix" default=""></xacro:arg>
+	<xacro:arg name="gz_odometry_frame" default="odom"></xacro:arg>
+	<xacro:property name="_ros2_control_pkg" value="$(arg ros2_control_pkg)"></xacro:property>
+	<xacro:property name="_ros2_control_path" value="$(find ${_ros2_control_pkg})"></xacro:property>
 	<xacro:include filename="$(find transbot_description)/urdf/shelf_lifter/__all__.urdf.xacro"></xacro:include>
 	<xacro:include filename="$(find transbot_gazebo)/urdf/shelf_lifter/mobilebase.urdf.xacro"></xacro:include>
+	<xacro:include filename="$(find transbot_gazebo)/urdf/shelf_lifter/__extras__.urdf.xacro"></xacro:include>
 	<gazebo>
 		<plugin filename="gz_ros2_control-system" name="gz_ros2_control::GazeboSimROS2ControlPlugin">
-			<parameters>$(find transbot_gazebo)/config/$(arg ros2_control_dict)</parameters>
+			<parameters>${_ros2_control_path}/config/$(arg ros2_control_dict)</parameters>
 			<ros>
 				<namespace>$(arg ros2_control_namespace)</namespace>
 			</ros>
+		</plugin>
+	</gazebo>
+	<gazebo>
+		<plugin filename="gz-sim-odometry-publisher-system" name="gz::sim::systems::OdometryPublisher">
+			<odom_frame>$(arg gz_odometry_frame_prefix)/$(arg gz_odometry_frame)</odom_frame>
+			<robot_base_frame>$(arg gz_odometry_frame_prefix)/gz_gtruth</robot_base_frame>
+			<odom_topic>/model/$(arg robot_name)/ground_truth/odometry</odom_topic>
+			<tf_topic>/model/$(arg robot_name)/ground_truth/pose</tf_topic>
+			<odom_publish_rate>50</odom_publish_rate>
+			<dimensions>3</dimensions>
+			<gaussian_noise>0.0</gaussian_noise>
 		</plugin>
 	</gazebo>

File: robotics/transbot-ros2ws/src/transbot_gazebo/urdf/shelf_lifter/mobilebase/castor/__all__.urdf.xacro (robot description, xacro)
@@ -1,14 +1,32 @@
 <?xml version="1.0" encoding="utf-8"?>
 <robot xmlns:xacro="http://www.ros.org/wiki/xacro" name="castor">
+	<xacro:arg name="robot_name" default="transbot"></xacro:arg>
 	<xacro:arg name="ros2_control_namespace" default="/transbot"></xacro:arg>
-	<xacro:arg name="ros2_control_dict" default="shelf_lifter/mobilebase/ros2_control.yaml"></xacro:arg>
+	<xacro:arg name="ros2_control_dict" default="shelf_lifter/mobilebase.yaml"></xacro:arg>
+	<xacro:arg name="ros2_control_pkg" default="transbot_controller"></xacro:arg>
+	<xacro:arg name="gz_odometry_frame_prefix" default=""></xacro:arg>
+	<xacro:arg name="gz_odometry_frame" default="odom"></xacro:arg>
+	<xacro:property name="_ros2_control_pkg" value="$(arg ros2_control_pkg)"></xacro:property>
+	<xacro:property name="_ros2_control_path" value="$(find ${_ros2_control_pkg})"></xacro:property>
 	<xacro:include filename="$(find transbot_description)/urdf/shelf_lifter/mobilebase/__all__.urdf.xacro"></xacro:include>
 	<xacro:include filename="$(find transbot_gazebo)/urdf/shelf_lifter/mobilebase/castor.urdf.xacro"></xacro:include>
+	<xacro:include filename="$(find transbot_gazebo)/urdf/shelf_lifter/mobilebase/__extras__.urdf.xacro"></xacro:include>
 	<gazebo>
 		<plugin filename="gz_ros2_control-system" name="gz_ros2_control::GazeboSimROS2ControlPlugin">
-			<parameters>$(find transbot_gazebo)/config/$(arg ros2_control_dict)</parameters>
+			<parameters>${_ros2_control_path}/config/$(arg ros2_control_dict)</parameters>
 			<ros>
 				<namespace>$(arg ros2_control_namespace)</namespace>
 			</ros>
+		</plugin>
+	</gazebo>
+	<gazebo>
+		<plugin filename="gz-sim-odometry-publisher-system" name="gz::sim::systems::OdometryPublisher">
+			<odom_frame>$(arg gz_odometry_frame_prefix)/$(arg gz_odometry_frame)</odom_frame>
+			<robot_base_frame>$(arg gz_odometry_frame_prefix)/gz_gtruth</robot_base_frame>
+			<odom_topic>/model/$(arg robot_name)/ground_truth/odometry</odom_topic>
+			<tf_topic>/model/$(arg robot_name)/ground_truth/pose</tf_topic>
+			<odom_publish_rate>50</odom_publish_rate>
+			<dimensions>3</dimensions>
+			<gaussian_noise>0.0</gaussian_noise>
 		</plugin>
 	</gazebo>

File: robotics/transbot-ros2ws/src/transbot_gazebo/urdf/shelf_lifter/mobilebase/doublebar/__all__.urdf.xacro (robot description, xacro)
@@ -1,14 +1,32 @@
 <?xml version="1.0" encoding="utf-8"?>
 <robot xmlns:xacro="http://www.ros.org/wiki/xacro" name="doublebar">
+	<xacro:arg name="robot_name" default="transbot"></xacro:arg>
 	<xacro:arg name="ros2_control_namespace" default="/transbot"></xacro:arg>
-	<xacro:arg name="ros2_control_dict" default="shelf_lifter/mobilebase/ros2_control.yaml"></xacro:arg>
+	<xacro:arg name="ros2_control_dict" default="shelf_lifter/mobilebase.yaml"></xacro:arg>
+	<xacro:arg name="ros2_control_pkg" default="transbot_controller"></xacro:arg>
+	<xacro:arg name="gz_odometry_frame_prefix" default=""></xacro:arg>
+	<xacro:arg name="gz_odometry_frame" default="odom"></xacro:arg>
+	<xacro:property name="_ros2_control_pkg" value="$(arg ros2_control_pkg)"></xacro:property>
+	<xacro:property name="_ros2_control_path" value="$(find ${_ros2_control_pkg})"></xacro:property>
 	<xacro:include filename="$(find transbot_description)/urdf/shelf_lifter/mobilebase/__all__.urdf.xacro"></xacro:include>
 	<xacro:include filename="$(find transbot_gazebo)/urdf/shelf_lifter/mobilebase/doublebar.urdf.xacro"></xacro:include>
+	<xacro:include filename="$(find transbot_gazebo)/urdf/shelf_lifter/mobilebase/__extras__.urdf.xacro"></xacro:include>
 	<gazebo>
 		<plugin filename="gz_ros2_control-system" name="gz_ros2_control::GazeboSimROS2ControlPlugin">
-			<parameters>$(find transbot_gazebo)/config/$(arg ros2_control_dict)</parameters>
+			<parameters>${_ros2_control_path}/config/$(arg ros2_control_dict)</parameters>
 			<ros>
 				<namespace>$(arg ros2_control_namespace)</namespace>
 			</ros>
+		</plugin>
+	</gazebo>
+	<gazebo>
+		<plugin filename="gz-sim-odometry-publisher-system" name="gz::sim::systems::OdometryPublisher">
+			<odom_frame>$(arg gz_odometry_frame_prefix)/$(arg gz_odometry_frame)</odom_frame>
+			<robot_base_frame>$(arg gz_odometry_frame_prefix)/gz_gtruth</robot_base_frame>
+			<odom_topic>/model/$(arg robot_name)/ground_truth/odometry</odom_topic>
+			<tf_topic>/model/$(arg robot_name)/ground_truth/pose</tf_topic>
+			<odom_publish_rate>50</odom_publish_rate>
+			<dimensions>3</dimensions>
+			<gaussian_noise>0.0</gaussian_noise>
 		</plugin>
 	</gazebo>

File: robotics/transbot-ros2ws/src/transbot_gazebo/urdf/shelf_lifter/mobilebase/doublebar/diff/__all__.urdf.xacro (robot description, xacro)
@@ -1,14 +1,32 @@
 <?xml version="1.0" encoding="utf-8"?>
 <robot xmlns:xacro="http://www.ros.org/wiki/xacro" name="diff">
+	<xacro:arg name="robot_name" default="transbot"></xacro:arg>
 	<xacro:arg name="ros2_control_namespace" default="/transbot"></xacro:arg>
-	<xacro:arg name="ros2_control_dict" default="shelf_lifter/mobilebase/doublebar/ros2_control.yaml"></xacro:arg>
+	<xacro:arg name="ros2_control_dict" default="shelf_lifter/mobilebase/doublebar.yaml"></xacro:arg>
+	<xacro:arg name="ros2_control_pkg" default="transbot_controller"></xacro:arg>
+	<xacro:arg name="gz_odometry_frame_prefix" default=""></xacro:arg>
+	<xacro:arg name="gz_odometry_frame" default="odom"></xacro:arg>
+	<xacro:property name="_ros2_control_pkg" value="$(arg ros2_control_pkg)"></xacro:property>
+	<xacro:property name="_ros2_control_path" value="$(find ${_ros2_control_pkg})"></xacro:property>
 	<xacro:include filename="$(find transbot_description)/urdf/shelf_lifter/mobilebase/doublebar/__all__.urdf.xacro"></xacro:include>
 	<xacro:include filename="$(find transbot_gazebo)/urdf/shelf_lifter/mobilebase/doublebar/diff.urdf.xacro"></xacro:include>
+	<xacro:include filename="$(find transbot_gazebo)/urdf/shelf_lifter/mobilebase/doublebar/__extras__.urdf.xacro"></xacro:include>
 	<gazebo>
 		<plugin filename="gz_ros2_control-system" name="gz_ros2_control::GazeboSimROS2ControlPlugin">
-			<parameters>$(find transbot_gazebo)/config/$(arg ros2_control_dict)</parameters>
+			<parameters>${_ros2_control_path}/config/$(arg ros2_control_dict)</parameters>
 			<ros>
 				<namespace>$(arg ros2_control_namespace)</namespace>
 			</ros>
+		</plugin>
+	</gazebo>
+	<gazebo>
+		<plugin filename="gz-sim-odometry-publisher-system" name="gz::sim::systems::OdometryPublisher">
+			<odom_frame>$(arg gz_odometry_frame_prefix)/$(arg gz_odometry_frame)</odom_frame>
+			<robot_base_frame>$(arg gz_odometry_frame_prefix)/gz_gtruth</robot_base_frame>
+			<odom_topic>/model/$(arg robot_name)/ground_truth/odometry</odom_topic>
+			<tf_topic>/model/$(arg robot_name)/ground_truth/pose</tf_topic>
+			<odom_publish_rate>50</odom_publish_rate>
+			<dimensions>3</dimensions>
+			<gaussian_noise>0.0</gaussian_noise>
 		</plugin>
 	</gazebo>
