Commit message: Modified SixWheels Robot with Castor Prismatic Suspensions

File: robotics/transbot-ros2ws/src/transbot_description/urdf/mobilebase_diffdrive_6wheels_ltype_csuspp/camera.urdf.xacro (robot description, xacro)
@@ -4,7 +4,7 @@
 		<link name="${prefix}${name}${suffix}">
 			<inertial density="2000">
-				<origin xyz="0.0015456753955469056 -7.860687397225977e-12 1.8865649753342346e-11" rpy="0 0 0"></origin>
+				<origin xyz="0.0015456753955469056 -7.860687397225977e-12 -2.096183305926927e-12" rpy="0 0 0"></origin>
 				<mass value="0.2824747934937477"></mass>
-				<inertia ixx="0.0002409766617953816" ixy="-7.916904363093267e-13" ixz="-1.4349346685098745e-13" iyy="0.00015319900510290196" iyz="-1.8503717495987516e-15" izz="0.000279198877682898"></inertia>
+				<inertia ixx="0.0002409766617953816" ixy="-7.916904363093267e-13" ixz="2.498998022112951e-14" iyy="0.00015319900510290196" iyz="-1.8503717030541324e-15" izz="0.000279198877682898"></inertia>
 			</inertial>
 			<visual>

File: robotics/transbot-ros2ws/src/transbot_description/urdf/mobilebase_diffdrive_6wheels_ltype_csuspp/castor/arm.urdf.xacro (robot description, xacro)
@@ -4,7 +4,7 @@
 		<link name="${prefix}${name}${suffix}">
 			<inertial density="7850">
-				<origin xyz="0.023216223476559487 -5.499152560757377e-09 -0.023419604856066874" rpy="0 0 0"></origin>
+				<origin xyz="0.023216224918960162 -1.1854730520321233e-08 -0.023419606298467545" rpy="0 0 0"></origin>
 				<mass value="0.006568149425826657"></mass>
-				<inertia ixx="7.06487723744569e-06" ixy="-7.469593134069236e-13" ixz="1.2443357829905416e-06" iyy="4.505877976838242e-06" iyz="-2.7216179554656136e-12" izz="6.2024474186650775e-06"></inertia>
+				<inertia ixx="7.064875372609343e-06" ixy="-1.7133308560602608e-12" ixz="1.2443353411672071e-06" iyy="4.505877093191572e-06" iyz="-1.3739064829533716e-12" izz="6.202445557682362e-06"></inertia>
 			</inertial>
 			<visual>

File: robotics/transbot-ros2ws/src/transbot_description/urdf/mobilebase_diffdrive_6wheels_ltype_csuspp/castor/wheel.urdf.xacro (robot description, xacro)
@@ -4,7 +4,7 @@
 		<link name="${prefix}${name}${suffix}">
 			<inertial density="2500">
-				<origin xyz="-2.269997773998308e-10 4.981912077029785e-09 1.3228093841629953e-09" rpy="0 0 0"></origin>
-				<mass value="0.4594143247231841"></mass>
-				<inertia ixx="0.0004709492562445302" ixy="2.9647001926053876e-11" ixz="2.766305565072593e-12" iyy="0.00047094983225785266" iyz="-6.898645291669016e-12" izz="0.0008008165423234345"></inertia>
+				<origin xyz="-2.082552054383188e-09 -4.39983728040884e-10 -1.620738302486742e-10" rpy="0 0 0"></origin>
+				<mass value="0.4594138202567895"></mass>
+				<inertia ixx="0.00047094990046995605" ixy="1.4770361281276227e-11" ixz="1.1657343309210693e-12" iyy="0.00047094917287419274" iyz="-9.76996228909408e-13" izz="0.0008008168151718543"></inertia>
 			</inertial>
 			<visual>

File: robotics/transbot-ros2ws/src/transbot_description/urdf/mobilebase_diffdrive_6wheels_ltype_csuspp/doublebar/diff/wheel.urdf.xacro (robot description, xacro)
@@ -4,7 +4,7 @@
 		<link name="${prefix}${name}${suffix}">
 			<inertial density="2500">
-				<origin xyz="1.5806070609371153e-09 1.4316135311553461e-09 1.5819836565310336e-09" rpy="0 0 0"></origin>
-				<mass value="0.40324951987713575"></mass>
-				<inertia ixx="0.0003983033404134991" ixy="-1.6095911767625574e-12" ixz="-1.0528604933629682e-12" iyy="0.0003983025825012475" iyz="-6.207533573160245e-12" izz="0.0006993442790796186"></inertia>
+				<origin xyz="-4.629070430847593e-09 -2.0538772661327532e-10 -1.500486742684116e-09" rpy="0 0 0"></origin>
+				<mass value="0.4032501795639594"></mass>
+				<inertia ixx="0.0003983030675650895" ixy="6.911023063451691e-12" ixz="-4.118924620440517e-12" iyy="0.00039830203680441884" iyz="-2.1302403042252493e-12" izz="0.0006993443700290819"></inertia>
 			</inertial>
 			<visual>

File: robotics/transbot-ros2ws/src/transbot_description/urdf/mobilebase_diffdrive_6wheels_ltype_csuspp/mobilebase_diffdrive_6wheels_ltype_csuspp.urdf.xacro (robot description, xacro)
@@ -9,4 +9,5 @@
 		<xacro:include filename="$(find transbot_description)/urdf/mobilebase_diffdrive_6wheels_ltype_csuspp/camera.urdf.xacro"></xacro:include>
 		<xacro:include filename="$(find transbot_description)/urdf/mobilebase_diffdrive_6wheels_ltype_csuspp/lidar.urdf.xacro"></xacro:include>
+		<xacro:include filename="$(find transbot_description)/urdf/mobilebase_diffdrive_6wheels_ltype_csuspp/imu.urdf.xacro"></xacro:include>
 		<joint name="j/${prefix}${name}${suffix}chassis" type="fixed">
 			<origin xyz="0.0 0.0 0.13" rpy="0.0 0.0 0.0"></origin>
@@ -26,5 +27,5 @@
 			<parent link="${prefix}${name}${suffix}_"></parent>
 			<child link="${prefix}${name}${suffix}castor0/_"></child>
-			<dynamics damping="0.0" friction="0.0"></dynamics>
+			<dynamics damping="10" friction="10"></dynamics>
 			<axis xyz="0 0 1"></axis>
 			<limit lower="-0.05" upper="0.05" effort="1000000.0" velocity="1000000.0"></limit>
@@ -34,5 +35,5 @@
 			<parent link="${prefix}${name}${suffix}_"></parent>
 			<child link="${prefix}${name}${suffix}castor1/_"></child>
-			<dynamics damping="0.0" friction="0.0"></dynamics>
+			<dynamics damping="10" friction="10"></dynamics>
 			<axis xyz="0 0 1"></axis>
 			<limit lower="-0.05" upper="0.05" effort="1000000.0" velocity="1000000.0"></limit>
@@ -42,5 +43,5 @@
 			<parent link="${prefix}${name}${suffix}_"></parent>
 			<child link="${prefix}${name}${suffix}castor2/_"></child>
-			<dynamics damping="0.0" friction="0.0"></dynamics>
+			<dynamics damping="10" friction="10"></dynamics>
 			<axis xyz="0 0 1"></axis>
 			<limit lower="-0.05" upper="0.05" effort="1000000.0" velocity="1000000.0"></limit>
@@ -50,5 +51,5 @@
 			<parent link="${prefix}${name}${suffix}_"></parent>
 			<child link="${prefix}${name}${suffix}castor3/_"></child>
-			<dynamics damping="0.0" friction="0.0"></dynamics>
+			<dynamics damping="10" friction="10"></dynamics>
 			<axis xyz="0 0 1"></axis>
 			<limit lower="-0.05" upper="0.05" effort="1000000.0" velocity="1000000.0"></limit>
@@ -72,4 +73,9 @@
 			<child link="${prefix}${name}${suffix}lidar"></child>
 		</joint>
+		<joint name="j/${prefix}${name}${suffix}imu" type="fixed">
+			<origin xyz="0.3 -0.25 0.17" rpy="0.0 0.0 0.0"></origin>
+			<parent link="${prefix}${name}${suffix}_"></parent>
+			<child link="${prefix}${name}${suffix}imu"></child>
+		</joint>
 		<xacro:chassis prefix="${prefix}${name}${suffix}" suffix=""></xacro:chassis>
 		<xacro:control prefix="${prefix}${name}${suffix}" suffix=""></xacro:control>
@@ -81,4 +87,5 @@
 		<xacro:camera prefix="${prefix}${name}${suffix}" suffix=""></xacro:camera>
 		<xacro:lidar prefix="${prefix}${name}${suffix}" suffix=""></xacro:lidar>
+		<xacro:imu prefix="${prefix}${name}${suffix}" suffix=""></xacro:imu>
 	</xacro:macro>
 </robot>

File: robotics/transbot-ros2ws/src/transbot_gazebo/urdf/mobilebase_diffdrive_6wheels_ltype_csuspp/mobilebase_diffdrive_6wheels_ltype_csuspp.urdf.xacro (robot description, xacro)
@@ -17,7 +17,4 @@
 			<state_interface name="velocity"></state_interface>
 			<state_interface name="effort"></state_interface>
-			<command_interface name="position"></command_interface>
-			<command_interface name="velocity"></command_interface>
-			<command_interface name="effort"></command_interface>
 		</joint>
 		<joint name="j/${prefix}${name}${suffix}castor1/_">
@@ -27,7 +24,4 @@
 			<state_interface name="velocity"></state_interface>
 			<state_interface name="effort"></state_interface>
-			<command_interface name="position"></command_interface>
-			<command_interface name="velocity"></command_interface>
-			<command_interface name="effort"></command_interface>
 		</joint>
 		<joint name="j/${prefix}${name}${suffix}castor2/_">
@@ -37,7 +31,4 @@
 			<state_interface name="velocity"></state_interface>
 			<state_interface name="effort"></state_interface>
-			<command_interface name="position"></command_interface>
-			<command_interface name="velocity"></command_interface>
-			<command_interface name="effort"></command_interface>
 		</joint>
 		<joint name="j/${prefix}${name}${suffix}castor3/_">
@@ -47,7 +38,4 @@
 			<state_interface name="velocity"></state_interface>
 			<state_interface name="effort"></state_interface>
-			<command_interface name="position"></command_interface>
-			<command_interface name="velocity"></command_interface>
-			<command_interface name="effort"></command_interface>
 		</joint>
 		<joint name="j/${prefix}${name}${suffix}control">
@@ -73,20 +61,20 @@
 		<gazebo reference="j/${prefix}${name}${suffix}castor0/_">
 			<implicitSpringDamper>true</implicitSpringDamper>
-			<springStiffness>0.5</springStiffness>
+			<springStiffness>3000</springStiffness>
 			<springReference>0.0</springReference>
 		</gazebo>
 		<gazebo reference="j/${prefix}${name}${suffix}castor1/_">
 			<implicitSpringDamper>true</implicitSpringDamper>
-			<springStiffness>0.5</springStiffness>
+			<springStiffness>3000</springStiffness>
 			<springReference>0.0</springReference>
 		</gazebo>
 		<gazebo reference="j/${prefix}${name}${suffix}castor2/_">
 			<implicitSpringDamper>true</implicitSpringDamper>
-			<springStiffness>0.5</springStiffness>
+			<springStiffness>3000</springStiffness>
 			<springReference>0.0</springReference>
 		</gazebo>
 		<gazebo reference="j/${prefix}${name}${suffix}castor3/_">
 			<implicitSpringDamper>true</implicitSpringDamper>
-			<springStiffness>0.5</springStiffness>
+			<springStiffness>3000</springStiffness>
 			<springReference>0.0</springReference>
 		</gazebo>
