Commit message: Exported sixwheels and added cameras

File: robotics/transbot-ros2ws/src/transbot_description/urdf/mobilebase_diffdrive_6wheels_ltype/castor/arm.urdf.xacro (robot description, xacro)
@@ -4,7 +4,7 @@
 		<link name="${prefix}${name}${suffix}">
 			<inertial density="7850">
-				<origin xyz="0.023216223476559487 -1.1854730520321233e-08 -0.023419604856066874" rpy="0 0 0"></origin>
+				<origin xyz="0.023216224918960162 -1.1854730520321233e-08 -0.023419614952871575" rpy="0 0 0"></origin>
 				<mass value="0.006568149425826657"></mass>
-				<inertia ixx="7.064875816359493e-06" ixy="-1.7161063013112547e-12" ixz="1.2443357829905416e-06" iyy="4.505877976838242e-06" iyz="-1.3739065952639405e-12" izz="6.202445997578881e-06"></inertia>
+				<inertia ixx="7.06487271010787e-06" ixy="-1.7133308560602608e-12" ixz="1.2443340214776094e-06" iyy="4.505874430690099e-06" iyz="-1.3739058090899594e-12" izz="6.202445557682362e-06"></inertia>
 			</inertial>
 			<visual>

File: robotics/transbot-ros2ws/src/transbot_description/urdf/mobilebase_diffdrive_6wheels_ltype/castor/castor.urdf.xacro (robot description, xacro)
@@ -22,4 +22,5 @@
 			</collision>
 		</link>
+		<xacro:include filename="$(find transbot_description)/urdf/mobilebase_diffdrive_6wheels_ltype/castor/__extras__.urdf.xacro"></xacro:include>
 		<xacro:include filename="$(find transbot_description)/urdf/mobilebase_diffdrive_6wheels_ltype/castor/arm.urdf.xacro"></xacro:include>
 		<xacro:include filename="$(find transbot_description)/urdf/mobilebase_diffdrive_6wheels_ltype/castor/wheel.urdf.xacro"></xacro:include>
@@ -36,4 +37,5 @@
 			<axis xyz="0 0 1"></axis>
 		</joint>
+		<xacro:castor-extras-description prefix="${prefix}${name}${suffix}"></xacro:castor-extras-description>
 		<xacro:arm prefix="${prefix}${name}${suffix}" suffix=""></xacro:arm>
 		<xacro:wheel prefix="${prefix}${name}${suffix}" suffix=""></xacro:wheel>

File: robotics/transbot-ros2ws/src/transbot_description/urdf/mobilebase_diffdrive_6wheels_ltype/castor/wheel.urdf.xacro (robot description, xacro)
@@ -4,7 +4,7 @@
 		<link name="${prefix}${name}${suffix}">
 			<inertial density="2500">
-				<origin xyz="9.976856274851814e-10 -1.6634337912257626e-11 1.3427357449894444e-10" rpy="0 0 0"></origin>
-				<mass value="0.49389704751471675"></mass>
-				<inertia ixx="0.000539365805707348" ixy="-6.631038319233847e-12" ixz="1.3026617483906892e-12" iyy="0.0005393657147578773" iyz="-1.1031447436551255e-21" izz="0.0009120414385203423"></inertia>
+				<origin xyz="-9.396248125394537e-09 -1.2619517440154898e-09 4.1001751417329526e-10" rpy="0 0 0"></origin>
+				<mass value="0.45941413069764775"></mass>
+				<inertia ixx="0.0004709500368941606" ixy="-2.6784075993538147e-12" ixz="-1.0362258558264331e-13" iyy="0.00047095012784359095" iyz="1.8108197747451987e-12" izz="0.0008008173911851263"></inertia>
 			</inertial>
 			<visual>

File: robotics/transbot-ros2ws/src/transbot_description/urdf/mobilebase_diffdrive_6wheels_ltype/chassis.urdf.xacro (robot description, xacro)
@@ -4,7 +4,7 @@
 		<link name="${prefix}${name}${suffix}">
 			<inertial density="7850">
-				<origin xyz="-0.11609746575277051 -0.00026483609977699 0.24375729246905095" rpy="0 0 0"></origin>
-				<mass value="3.7706432243188224"></mass>
-				<inertia ixx="0.26229166671580284" ixy="-0.00021814183586693777" ixz="0.08820158966257266" iyy="0.38611388218655324" iyz="-7.276365055565556e-05" izz="0.4149797591892294"></inertia>
+				<origin xyz="-0.08710447351018899 -5.427290924626776e-08 0.23152132526298272" rpy="0 0 0"></origin>
+				<mass value="3.7537477910518646"></mass>
+				<inertia ixx="0.24047775252227827" ixy="1.7745516803445148e-08" ixz="0.05998296526638469" iyy="0.31535036791706106" iyz="1.313363916849617e-07" izz="0.3762323023952737"></inertia>
 			</inertial>
 			<visual>

File: robotics/transbot-ros2ws/src/transbot_description/urdf/mobilebase_diffdrive_6wheels_ltype/doublebar/diff/diff.urdf.xacro (robot description, xacro)
@@ -22,4 +22,5 @@
 			</collision>
 		</link>
+		<xacro:include filename="$(find transbot_description)/urdf/mobilebase_diffdrive_6wheels_ltype/doublebar/diff/__extras__.urdf.xacro"></xacro:include>
 		<xacro:include filename="$(find transbot_description)/urdf/mobilebase_diffdrive_6wheels_ltype/doublebar/diff/wheel.urdf.xacro"></xacro:include>
 		<joint name="j/${prefix}${name}${suffix}wheel0" type="continuous">
@@ -35,4 +36,5 @@
 			<axis xyz="0 0 1"></axis>
 		</joint>
+		<xacro:diff-extras-description prefix="${prefix}${name}${suffix}"></xacro:diff-extras-description>
 		<xacro:wheel prefix="${prefix}${name}${suffix}" suffix="0"></xacro:wheel>
 		<xacro:wheel prefix="${prefix}${name}${suffix}" suffix="1"></xacro:wheel>

File: robotics/transbot-ros2ws/src/transbot_description/urdf/mobilebase_diffdrive_6wheels_ltype/doublebar/diff/wheel.urdf.xacro (robot description, xacro)
@@ -4,7 +4,7 @@
 		<link name="${prefix}${name}${suffix}">
 			<inertial density="2500">
-				<origin xyz="2.6436662400850254e-10 1.2846341067506226e-10 -2.1101985721945073e-10" rpy="0 0 0"></origin>
-				<mass value="0.43773395009338856"></mass>
-				<inertia ixx="0.0004636484770041231" ixy="-5.443562252749146e-12" ixz="-3.5527139229974206e-13" iyy="0.0004636485376371031" iyz="4.62581060690524e-16" izz="0.0008105680535663851"></inertia>
+				<origin xyz="5.747090891466626e-09 -8.817993841025995e-10 2.3049667826529517e-09" rpy="0 0 0"></origin>
+				<mass value="0.40325037358949584"></mass>
+				<inertia ixx="0.0003983029425095665" ixy="6.2618871117646805e-12" ixz="3.837676263586289e-12" iyy="0.0003983026090281628" iyz="7.75166885690447e-12" izz="0.0006993441578136466"></inertia>
 			</inertial>
 			<visual>

File: robotics/transbot-ros2ws/src/transbot_description/urdf/mobilebase_diffdrive_6wheels_ltype/doublebar/doublebar.urdf.xacro (robot description, xacro)
@@ -22,4 +22,5 @@
 			</collision>
 		</link>
+		<xacro:include filename="$(find transbot_description)/urdf/mobilebase_diffdrive_6wheels_ltype/doublebar/__extras__.urdf.xacro"></xacro:include>
 		<xacro:include filename="$(find transbot_description)/urdf/mobilebase_diffdrive_6wheels_ltype/doublebar/diff/diff.urdf.xacro"></xacro:include>
 		<joint name="j/${prefix}${name}${suffix}diff/_" type="revolute">
@@ -31,4 +32,5 @@
 			<limit lower="-5" upper="5" effort="1000000.0" velocity="1000000.0"></limit>
 		</joint>
+		<xacro:doublebar-extras-description prefix="${prefix}${name}${suffix}"></xacro:doublebar-extras-description>
 		<xacro:diff prefix="${prefix}${name}${suffix}" suffix="/"></xacro:diff>
 	</xacro:macro>

File: robotics/transbot-ros2ws/src/transbot_description/urdf/mobilebase_diffdrive_6wheels_ltype/mobilebase_diffdrive_6wheels_ltype.urdf.xacro (robot description, xacro)
@@ -3,8 +3,12 @@
 	<xacro:macro name="mobilebase_diffdrive_6wheels_ltype" params="prefix='' name='mobilebase_diffdrive_6wheels_ltype' suffix=''">
 		<link name="${prefix}${name}${suffix}_"></link>
+		<xacro:include filename="$(find transbot_description)/urdf/mobilebase_diffdrive_6wheels_ltype//__extras__.urdf.xacro"></xacro:include>
 		<xacro:include filename="$(find transbot_description)/urdf/mobilebase_diffdrive_6wheels_ltype/chassis.urdf.xacro"></xacro:include>
 		<xacro:include filename="$(find transbot_description)/urdf/mobilebase_diffdrive_6wheels_ltype/control.urdf.xacro"></xacro:include>
 		<xacro:include filename="$(find transbot_description)/urdf/mobilebase_diffdrive_6wheels_ltype/doublebar/doublebar.urdf.xacro"></xacro:include>
 		<xacro:include filename="$(find transbot_description)/urdf/mobilebase_diffdrive_6wheels_ltype/castor/castor.urdf.xacro"></xacro:include>
+		<xacro:include filename="$(find transbot_description)/urdf/mobilebase_diffdrive_6wheels_ltype/camera.urdf.xacro"></xacro:include>
+		<xacro:include filename="$(find transbot_description)/urdf/mobilebase_diffdrive_6wheels_ltype/lidar.urdf.xacro"></xacro:include>
+		<xacro:include filename="$(find transbot_description)/urdf/mobilebase_diffdrive_6wheels_ltype/imu.urdf.xacro"></xacro:include>
 		<joint name="j/${prefix}${name}${suffix}chassis" type="fixed">
 			<origin xyz="0.0 0.0 0.13" rpy="0.0 0.0 0.0"></origin>
@@ -41,11 +45,27 @@
 		</joint>
 		<joint name="j/${prefix}${name}${suffix}control" type="prismatic">
-			<origin xyz="0.075 0.0 0.17" rpy="0.0 0.0 1.5707963267948966"></origin>
+			<origin xyz="-0.075 0.0 0.17" rpy="0.0 0.0 1.5707963267948966"></origin>
 			<parent link="${prefix}${name}${suffix}_"></parent>
 			<child link="${prefix}${name}${suffix}control"></child>
 			<dynamics damping="10" friction="10"></dynamics>
-			<axis xyz="0 -1 0"></axis>
+			<axis xyz="0 1 0"></axis>
 			<limit lower="0.0" upper="0.5" effort="1000000.0" velocity="1000000.0"></limit>
 		</joint>
+		<joint name="j/${prefix}${name}${suffix}camera" type="fixed">
+			<origin xyz="-0.28 0.0 0.68" rpy="0.0 0.0 0.0"></origin>
+			<parent link="${prefix}${name}${suffix}_"></parent>
+			<child link="${prefix}${name}${suffix}camera"></child>
+		</joint>
+		<joint name="j/${prefix}${name}${suffix}lidar" type="fixed">
+			<origin xyz="0.3 0.0 0.17" rpy="0.0 0.0 0.0"></origin>
+			<parent link="${prefix}${name}${suffix}_"></parent>
+			<child link="${prefix}${name}${suffix}lidar"></child>
+		</joint>
+		<joint name="j/${prefix}${name}${suffix}imu" type="fixed">
+			<origin xyz="0.3 -0.25 0.17" rpy="0.0 0.0 0.0"></origin>
+			<parent link="${prefix}${name}${suffix}_"></parent>
+			<child link="${prefix}${name}${suffix}imu"></child>
+		</joint>
+		<xacro:mobilebase_diffdrive_6wheels_ltype-extras-description prefix="${prefix}${name}${suffix}"></xacro:mobilebase_diffdrive_6wheels_ltype-extras-description>
 		<xacro:chassis prefix="${prefix}${name}${suffix}" suffix=""></xacro:chassis>
 		<xacro:control prefix="${prefix}${name}${suffix}" suffix=""></xacro:control>
@@ -55,4 +75,7 @@
 		<xacro:castor prefix="${prefix}${name}${suffix}" suffix="2/"></xacro:castor>
 		<xacro:castor prefix="${prefix}${name}${suffix}" suffix="3/"></xacro:castor>
+		<xacro:camera prefix="${prefix}${name}${suffix}" suffix=""></xacro:camera>
+		<xacro:lidar prefix="${prefix}${name}${suffix}" suffix=""></xacro:lidar>
+		<xacro:imu prefix="${prefix}${name}${suffix}" suffix=""></xacro:imu>
 	</xacro:macro>
 </robot>

File: robotics/transbot-ros2ws/src/transbot_description/urdf/mobilebase_diffdrive_6wheels_ltype_csuspp/__extras__.urdf.xacro (robot description, xacro)
@@ -1,2 +1,6 @@
 <?xml version="1.0" encoding="utf-8"?>
-<robot xmlns:xacro="http://www.ros.org/wiki/xacro" name="mobilebase_diffdrive_6wheels_ltype_csuspp"></robot>
+<robot xmlns:xacro="http://www.ros.org/wiki/xacro" name="mobilebase_diffdrive_6wheels_ltype_csuspp">
+	<xacro:macro name="mobilebase_diffdrive_6wheels_ltype_csuspp-extras-description" params="prefix='' name='mobilebase_diffdrive_6wheels_ltype_csuspp' suffix=''">
+	<!-- THIS FILE SHOULD BE PERSISTENT-->
+	</xacro:macro>
+</robot>

File: robotics/transbot-ros2ws/src/transbot_description/urdf/mobilebase_diffdrive_6wheels_ltype_csuspp/camera.urdf.xacro (robot description, xacro)
@@ -4,7 +4,7 @@
 		<link name="${prefix}${name}${suffix}">
 			<inertial density="2000">
-				<origin xyz="0.0015456753955469056 -7.860687397225977e-12 -2.096183305926927e-12" rpy="0 0 0"></origin>
+				<origin xyz="0.0015456753955469056 1.0480916529634636e-12 -1.801407528530953e-12" rpy="0 0 0"></origin>
 				<mass value="0.2824747934937477"></mass>
-				<inertia ixx="0.0002409766617953816" ixy="-7.916904363093267e-13" ixz="2.498998022112951e-14" iyy="0.00015319900510290196" iyz="-1.8503717030541324e-15" izz="0.000279198877682898"></inertia>
+				<inertia ixx="0.0002409766617953816" ixy="-7.878007356404657e-13" ixz="3.0322853980014885e-14" iyy="0.00015319900510290196" iyz="-9.251858539076294e-15" izz="0.000279198877682898"></inertia>
 			</inertial>
 			<visual>

File: robotics/transbot-ros2ws/src/transbot_description/urdf/mobilebase_diffdrive_6wheels_ltype_csuspp/castor/__extras__.urdf.xacro (robot description, xacro)
@@ -1,2 +1,4 @@
 <?xml version="1.0" encoding="utf-8"?>
-<robot xmlns:xacro="http://www.ros.org/wiki/xacro" name="castor"></robot>
+<robot xmlns:xacro="http://www.ros.org/wiki/xacro" name="castor">
+	<xacro:macro name="castor-extras-description" params="prefix='' name='castor' suffix=''"></xacro:macro>
+</robot>

File: robotics/transbot-ros2ws/src/transbot_description/urdf/mobilebase_diffdrive_6wheels_ltype_csuspp/castor/arm.urdf.xacro (robot description, xacro)
@@ -4,7 +4,7 @@
 		<link name="${prefix}${name}${suffix}">
 			<inertial density="7850">
-				<origin xyz="0.023216224918960162 -1.1854730520321233e-08 -0.023419606298467545" rpy="0 0 0"></origin>
+				<origin xyz="0.023216224918960162 -5.499152560757377e-09 -0.023419614952871575" rpy="0 0 0"></origin>
 				<mass value="0.006568149425826657"></mass>
-				<inertia ixx="7.064875372609343e-06" ixy="-1.7133308560602608e-12" ixz="1.2443353411672071e-06" iyy="4.505877093191572e-06" iyz="-1.3739064829533716e-12" izz="6.202445557682362e-06"></inertia>
+				<inertia ixx="7.064874131194068e-06" ixy="-7.441838079437996e-13" ixz="1.2443340214776094e-06" iyy="4.505874430690099e-06" iyz="-2.7216175907765425e-12" izz="6.202446978768557e-06"></inertia>
 			</inertial>
 			<visual>

File: robotics/transbot-ros2ws/src/transbot_description/urdf/mobilebase_diffdrive_6wheels_ltype_csuspp/castor/castor.urdf.xacro (robot description, xacro)
@@ -22,4 +22,5 @@
 			</collision>
 		</link>
+		<xacro:include filename="$(find transbot_description)/urdf/mobilebase_diffdrive_6wheels_ltype_csuspp/castor/__extras__.urdf.xacro"></xacro:include>
 		<xacro:include filename="$(find transbot_description)/urdf/mobilebase_diffdrive_6wheels_ltype_csuspp/castor/arm.urdf.xacro"></xacro:include>
 		<xacro:include filename="$(find transbot_description)/urdf/mobilebase_diffdrive_6wheels_ltype_csuspp/castor/wheel.urdf.xacro"></xacro:include>
@@ -36,4 +37,5 @@
 			<axis xyz="0 0 1"></axis>
 		</joint>
+		<xacro:castor-extras-description prefix="${prefix}${name}${suffix}"></xacro:castor-extras-description>
 		<xacro:arm prefix="${prefix}${name}${suffix}" suffix=""></xacro:arm>
 		<xacro:wheel prefix="${prefix}${name}${suffix}" suffix=""></xacro:wheel>

File: robotics/transbot-ros2ws/src/transbot_description/urdf/mobilebase_diffdrive_6wheels_ltype_csuspp/castor/wheel.urdf.xacro (robot description, xacro)
@@ -4,7 +4,7 @@
 		<link name="${prefix}${name}${suffix}">
 			<inertial density="2500">
-				<origin xyz="-2.082552054383188e-09 -4.39983728040884e-10 -1.620738302486742e-10" rpy="0 0 0"></origin>
-				<mass value="0.4594138202567895"></mass>
-				<inertia ixx="0.00047094990046995605" ixy="1.4770361281276227e-11" ixz="1.1657343309210693e-12" iyy="0.00047094917287419274" iyz="-9.76996228909408e-13" izz="0.0008008168151718543"></inertia>
+				<origin xyz="1.4346420576654419e-08 -4.011565232160889e-11 1.3321940925597749e-09" rpy="0 0 0"></origin>
+				<mass value="0.4594142471129696"></mass>
+				<inertia ixx="0.0004709499459446904" ixy="-7.121282756611456e-11" ixz="4.781369273143673e-12" iyy="0.0004709498549951257" iyz="-1.096021424223687e-11" izz="0.0008008174518180531"></inertia>
 			</inertial>
 			<visual>

File: robotics/transbot-ros2ws/src/transbot_description/urdf/mobilebase_diffdrive_6wheels_ltype_csuspp/doublebar/__extras__.urdf.xacro (robot description, xacro)
@@ -1,2 +1,4 @@
 <?xml version="1.0" encoding="utf-8"?>
-<robot xmlns:xacro="http://www.ros.org/wiki/xacro" name="doublebar"></robot>
+<robot xmlns:xacro="http://www.ros.org/wiki/xacro" name="doublebar">
+	<xacro:macro name="doublebar-extras-description" params="prefix='' name='doublebar' suffix=''"></xacro:macro>
+</robot>

File: robotics/transbot-ros2ws/src/transbot_description/urdf/mobilebase_diffdrive_6wheels_ltype_csuspp/doublebar/diff/__extras__.urdf.xacro (robot description, xacro)
@@ -1,2 +1,4 @@
 <?xml version="1.0" encoding="utf-8"?>
-<robot xmlns:xacro="http://www.ros.org/wiki/xacro" name="diff"></robot>
+<robot xmlns:xacro="http://www.ros.org/wiki/xacro" name="diff">
+	<xacro:macro name="diff-extras-description" params="prefix='' name='diff' suffix=''"></xacro:macro>
+</robot>

File: robotics/transbot-ros2ws/src/transbot_description/urdf/mobilebase_diffdrive_6wheels_ltype_csuspp/doublebar/diff/diff.urdf.xacro (robot description, xacro)
@@ -22,4 +22,5 @@
 			</collision>
 		</link>
+		<xacro:include filename="$(find transbot_description)/urdf/mobilebase_diffdrive_6wheels_ltype_csuspp/doublebar/diff/__extras__.urdf.xacro"></xacro:include>
 		<xacro:include filename="$(find transbot_description)/urdf/mobilebase_diffdrive_6wheels_ltype_csuspp/doublebar/diff/wheel.urdf.xacro"></xacro:include>
 		<joint name="j/${prefix}${name}${suffix}wheel0" type="continuous">
@@ -35,4 +36,5 @@
 			<axis xyz="0 0 1"></axis>
 		</joint>
+		<xacro:diff-extras-description prefix="${prefix}${name}${suffix}"></xacro:diff-extras-description>
 		<xacro:wheel prefix="${prefix}${name}${suffix}" suffix="0"></xacro:wheel>
 		<xacro:wheel prefix="${prefix}${name}${suffix}" suffix="1"></xacro:wheel>

File: robotics/transbot-ros2ws/src/transbot_description/urdf/mobilebase_diffdrive_6wheels_ltype_csuspp/doublebar/diff/wheel.urdf.xacro (robot description, xacro)
@@ -4,7 +4,7 @@
 		<link name="${prefix}${name}${suffix}">
 			<inertial density="2500">
-				<origin xyz="-4.629070430847593e-09 -2.0538772661327532e-10 -1.500486742684116e-09" rpy="0 0 0"></origin>
-				<mass value="0.4032501795639594"></mass>
-				<inertia ixx="0.0003983030675650895" ixy="6.911023063451691e-12" ixz="-4.118924620440517e-12" iyy="0.00039830203680441884" iyz="-2.1302403042252493e-12" izz="0.0006993443700290819"></inertia>
+				<origin xyz="1.510424729166539e-08 2.220122359881174e-09 -2.5526612008389246e-09" rpy="0 0 0"></origin>
+				<mass value="0.40325045119971037"></mass>
+				<inertia ixx="0.0003983034616794566" ixy="-7.547068379725054e-13" ixz="-2.980964368853438e-12" iyy="0.00039830273408360516" iyz="-1.896170692783488e-12" izz="0.0006993446731938973"></inertia>
 			</inertial>
 			<visual>

File: robotics/transbot-ros2ws/src/transbot_description/urdf/mobilebase_diffdrive_6wheels_ltype_csuspp/doublebar/doublebar.urdf.xacro (robot description, xacro)
@@ -22,4 +22,5 @@
 			</collision>
 		</link>
+		<xacro:include filename="$(find transbot_description)/urdf/mobilebase_diffdrive_6wheels_ltype_csuspp/doublebar/__extras__.urdf.xacro"></xacro:include>
 		<xacro:include filename="$(find transbot_description)/urdf/mobilebase_diffdrive_6wheels_ltype_csuspp/doublebar/diff/diff.urdf.xacro"></xacro:include>
 		<joint name="j/${prefix}${name}${suffix}diff/_" type="revolute">
@@ -31,4 +32,5 @@
 			<limit lower="-5" upper="5" effort="1000000.0" velocity="1000000.0"></limit>
 		</joint>
+		<xacro:doublebar-extras-description prefix="${prefix}${name}${suffix}"></xacro:doublebar-extras-description>
 		<xacro:diff prefix="${prefix}${name}${suffix}" suffix="/"></xacro:diff>
 	</xacro:macro>

File: robotics/transbot-ros2ws/src/transbot_description/urdf/mobilebase_diffdrive_6wheels_ltype_csuspp/mobilebase_diffdrive_6wheels_ltype_csuspp.urdf.xacro (robot description, xacro)
@@ -3,4 +3,5 @@
 	<xacro:macro name="mobilebase_diffdrive_6wheels_ltype_csuspp" params="prefix='' name='mobilebase_diffdrive_6wheels_ltype_csuspp' suffix=''">
 		<link name="${prefix}${name}${suffix}_"></link>
+		<xacro:include filename="$(find transbot_description)/urdf/mobilebase_diffdrive_6wheels_ltype_csuspp//__extras__.urdf.xacro"></xacro:include>
 		<xacro:include filename="$(find transbot_description)/urdf/mobilebase_diffdrive_6wheels_ltype_csuspp/chassis.urdf.xacro"></xacro:include>
 		<xacro:include filename="$(find transbot_description)/urdf/mobilebase_diffdrive_6wheels_ltype_csuspp/control.urdf.xacro"></xacro:include>
@@ -78,4 +79,5 @@
 			<child link="${prefix}${name}${suffix}imu"></child>
 		</joint>
+		<xacro:mobilebase_diffdrive_6wheels_ltype_csuspp-extras-description prefix="${prefix}${name}${suffix}"></xacro:mobilebase_diffdrive_6wheels_ltype_csuspp-extras-description>
 		<xacro:chassis prefix="${prefix}${name}${suffix}" suffix=""></xacro:chassis>
 		<xacro:control prefix="${prefix}${name}${suffix}" suffix=""></xacro:control>
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