Commit message: shelf lifter con camara

File: robotics/transbot-ros2ws/src/transbot_description/urdf/mobilebase_diffdrive_6wheels_ltype_csuspp/castor/arm.urdf.xacro (robot description, xacro)
@@ -4,7 +4,7 @@
 		<link name="${prefix}${name}${suffix}">
 			<inertial density="7850">
-				<origin xyz="0.023216224918960162 -5.499152560757377e-09 -0.023419614952871575" rpy="0 0 0"></origin>
+				<origin xyz="0.023216223476559487 -5.499152560757377e-09 -0.023419604856066874" rpy="0 0 0"></origin>
 				<mass value="0.006568149425826657"></mass>
-				<inertia ixx="7.064874131194068e-06" ixy="-7.441838079437996e-13" ixz="1.2443340214776094e-06" iyy="4.505874430690099e-06" iyz="-2.7216175907765425e-12" izz="6.202446978768557e-06"></inertia>
+				<inertia ixx="7.06487723744569e-06" ixy="-7.469593134069236e-13" ixz="1.2443357829905416e-06" iyy="4.505877976838242e-06" iyz="-2.7216179554656136e-12" izz="6.2024474186650775e-06"></inertia>
 			</inertial>
 			<visual>

File: robotics/transbot-ros2ws/src/transbot_description/urdf/mobilebase_diffdrive_6wheels_ltype_csuspp/castor/wheel.urdf.xacro (robot description, xacro)
@@ -4,7 +4,7 @@
 		<link name="${prefix}${name}${suffix}">
 			<inertial density="2500">
-				<origin xyz="1.4346420576654419e-08 -4.011565232160889e-11 1.3321940925597749e-09" rpy="0 0 0"></origin>
-				<mass value="0.4594142471129696"></mass>
-				<inertia ixx="0.0004709499459446904" ixy="-7.121282756611456e-11" ixz="4.781369273143673e-12" iyy="0.0004709498549951257" iyz="-1.096021424223687e-11" izz="0.0008008174518180531"></inertia>
+				<origin xyz="6.729928253995315e-09 2.418218061725748e-10 5.822411775534214e-10" rpy="0 0 0"></origin>
+				<mass value="0.45941397547721863"></mass>
+				<inertia ixx="0.00047094981709960837" ixy="1.3338405202687647e-11" ixz="-2.979080447543647e-13" iyy="0.0004709493926687267" iyz="-3.6341299692548287e-12" izz="0.0008008172396026965"></inertia>
 			</inertial>
 			<visual>

File: robotics/transbot-ros2ws/src/transbot_description/urdf/mobilebase_diffdrive_6wheels_ltype_csuspp/doublebar/diff/wheel.urdf.xacro (robot description, xacro)
@@ -4,7 +4,7 @@
 		<link name="${prefix}${name}${suffix}">
 			<inertial density="2500">
-				<origin xyz="1.510424729166539e-08 2.220122359881174e-09 -2.5526612008389246e-09" rpy="0 0 0"></origin>
-				<mass value="0.40325045119971037"></mass>
-				<inertia ixx="0.0003983034616794566" ixy="-7.547068379725054e-13" ixz="-2.980964368853438e-12" iyy="0.00039830273408360516" iyz="-1.896170692783488e-12" izz="0.0006993446731938973"></inertia>
+				<origin xyz="-1.3133179567360486e-08 1.405182760529961e-09 1.984867109345394e-09" rpy="0 0 0"></origin>
+				<mass value="0.40324955868224305"></mass>
+				<inertia ixx="0.0003983035033646326" ixy="1.0166166016838435e-11" ixz="-7.947451602155554e-13" iyy="0.0003983028060852925" iyz="6.365742392148256e-12" izz="0.000699344764143391"></inertia>
 			</inertial>
 			<visual>

File: robotics/transbot-ros2ws/src/transbot_description/urdf/shelf_lifter/__extras__.urdf.xacro (robot description, xacro)
@@ -1,2 +1,4 @@
 <?xml version="1.0" encoding="utf-8"?>
-<robot xmlns:xacro="http://www.ros.org/wiki/xacro" name="shelf_lifter"></robot>
+<robot xmlns:xacro="http://www.ros.org/wiki/xacro" name="shelf_lifter">
+	<xacro:macro name="shelf_lifter-extras-description" params="prefix='' name='shelf_lifter' suffix=''"></xacro:macro>
+</robot>

File: robotics/transbot-ros2ws/src/transbot_description/urdf/shelf_lifter/mobilebase/__extras__.urdf.xacro (robot description, xacro)
@@ -1,2 +1,4 @@
 <?xml version="1.0" encoding="utf-8"?>
-<robot xmlns:xacro="http://www.ros.org/wiki/xacro" name="mobilebase"></robot>
+<robot xmlns:xacro="http://www.ros.org/wiki/xacro" name="mobilebase">
+	<xacro:macro name="mobilebase-extras-description" params="prefix='' name='mobilebase' suffix=''"></xacro:macro>
+</robot>

File: robotics/transbot-ros2ws/src/transbot_description/urdf/shelf_lifter/mobilebase/castor/arm.urdf.xacro (robot description, xacro)
@@ -4,7 +4,7 @@
 		<link name="${prefix}${name}${suffix}">
 			<inertial density="7850">
-				<origin xyz="0.023216223476559487 -5.499152560757377e-09 -0.023419604856066874" rpy="0 0 0"></origin>
+				<origin xyz="0.023216224918960162 -1.1854730520321233e-08 -0.023419614952871575" rpy="0 0 0"></origin>
 				<mass value="0.006568149425826657"></mass>
-				<inertia ixx="7.06487723744569e-06" ixy="-7.469593134069236e-13" ixz="1.2443357829905416e-06" iyy="4.505877976838242e-06" iyz="-2.7216179554656136e-12" izz="6.2024474186650775e-06"></inertia>
+				<inertia ixx="7.06487271010787e-06" ixy="-1.7133308560602608e-12" ixz="1.2443340214776094e-06" iyy="4.505874430690099e-06" iyz="-1.3739058090899594e-12" izz="6.202445557682362e-06"></inertia>
 			</inertial>
 			<visual>

File: robotics/transbot-ros2ws/src/transbot_description/urdf/shelf_lifter/mobilebase/castor/castor.urdf.xacro (robot description, xacro)
@@ -22,4 +22,5 @@
 			</collision>
 		</link>
+		<xacro:include filename="$(find transbot_description)/urdf/shelf_lifter/mobilebase/castor/__extras__.urdf.xacro"></xacro:include>
 		<xacro:include filename="$(find transbot_description)/urdf/shelf_lifter/mobilebase/castor/arm.urdf.xacro"></xacro:include>
 		<xacro:include filename="$(find transbot_description)/urdf/shelf_lifter/mobilebase/castor/wheel.urdf.xacro"></xacro:include>
@@ -36,4 +37,5 @@
 			<axis xyz="0 0 1"></axis>
 		</joint>
+		<xacro:castor-extras-description prefix="${prefix}${name}${suffix}"></xacro:castor-extras-description>
 		<xacro:arm prefix="${prefix}${name}${suffix}" suffix=""></xacro:arm>
 		<xacro:wheel prefix="${prefix}${name}${suffix}" suffix=""></xacro:wheel>

File: robotics/transbot-ros2ws/src/transbot_description/urdf/shelf_lifter/mobilebase/castor/wheel.urdf.xacro (robot description, xacro)
@@ -4,7 +4,7 @@
 		<link name="${prefix}${name}${suffix}">
 			<inertial density="2500">
-				<origin xyz="1.4340148303551888e-09 -3.5090750499906038e-09 -2.852402266199148e-10" rpy="0 0 0"></origin>
+				<origin xyz="1.4340953839351436e-09 -3.507463978391508e-09 -2.852402266199148e-10" rpy="0 0 0"></origin>
 				<mass value="0.4594138978670041"></mass>
-				<inertia ixx="0.00047094974130837766" ixy="-1.5209132563311692e-11" ixz="1.9058826710217818e-12" iyy="0.00047094934719401157" iyz="-1.2603575130752765e-11" izz="0.0008008167848553598"></inertia>
+				<inertia ixx="0.00047094974130837766" ixy="-1.5205663115428158e-11" ixz="1.9058826710112255e-12" iyy="0.00047094934719401157" iyz="-1.260380642742735e-11" izz="0.0008008167848553598"></inertia>
 			</inertial>
 			<visual>

File: robotics/transbot-ros2ws/src/transbot_description/urdf/shelf_lifter/mobilebase/doublebar/diff/diff.urdf.xacro (robot description, xacro)
@@ -22,4 +22,5 @@
 			</collision>
 		</link>
+		<xacro:include filename="$(find transbot_description)/urdf/shelf_lifter/mobilebase/doublebar/diff/__extras__.urdf.xacro"></xacro:include>
 		<xacro:include filename="$(find transbot_description)/urdf/shelf_lifter/mobilebase/doublebar/diff/wheel.urdf.xacro"></xacro:include>
 		<joint name="j/${prefix}${name}${suffix}wheel0" type="continuous">
@@ -35,4 +36,5 @@
 			<axis xyz="0 0 1"></axis>
 		</joint>
+		<xacro:diff-extras-description prefix="${prefix}${name}${suffix}"></xacro:diff-extras-description>
 		<xacro:wheel prefix="${prefix}${name}${suffix}" suffix="0"></xacro:wheel>
 		<xacro:wheel prefix="${prefix}${name}${suffix}" suffix="1"></xacro:wheel>

File: robotics/transbot-ros2ws/src/transbot_description/urdf/shelf_lifter/mobilebase/doublebar/diff/wheel.urdf.xacro (robot description, xacro)
@@ -4,7 +4,7 @@
 		<link name="${prefix}${name}${suffix}">
 			<inertial density="2500">
-				<origin xyz="4.752325537276356e-09 -4.403267049900442e-10 1.1552381330584986e-09" rpy="0 0 0"></origin>
+				<origin xyz="4.750857169773262e-09 -4.447318074993235e-10 1.1552381330584986e-09" rpy="0 0 0"></origin>
 				<mass value="0.40324983031799394"></mass>
-				<inertia ixx="0.00039830266587159653" ixy="1.0545151870168692e-11" ixz="7.179444439778207e-12" iyy="0.0003983027871375477" iyz="-7.221077640592899e-13" izz="0.0006993444306620614"></inertia>
+				<inertia ixx="0.00039830266587159653" ixy="1.05451518619902e-11" ixz="7.1794444390941686e-12" iyy="0.0003983027871375477" iyz="-7.221077661114051e-13" izz="0.0006993444306620614"></inertia>
 			</inertial>
 			<visual>

File: robotics/transbot-ros2ws/src/transbot_description/urdf/shelf_lifter/mobilebase/doublebar/doublebar.urdf.xacro (robot description, xacro)
@@ -22,4 +22,5 @@
 			</collision>
 		</link>
+		<xacro:include filename="$(find transbot_description)/urdf/shelf_lifter/mobilebase/doublebar/__extras__.urdf.xacro"></xacro:include>
 		<xacro:include filename="$(find transbot_description)/urdf/shelf_lifter/mobilebase/doublebar/diff/diff.urdf.xacro"></xacro:include>
 		<joint name="j/${prefix}${name}${suffix}diff/_" type="revolute">
@@ -31,4 +32,5 @@
 			<limit lower="-5" upper="5" effort="1000000.0" velocity="1000000.0"></limit>
 		</joint>
+		<xacro:doublebar-extras-description prefix="${prefix}${name}${suffix}"></xacro:doublebar-extras-description>
 		<xacro:diff prefix="${prefix}${name}${suffix}" suffix="/"></xacro:diff>
 	</xacro:macro>

File: robotics/transbot-ros2ws/src/transbot_description/urdf/shelf_lifter/mobilebase/mobilebase.urdf.xacro (robot description, xacro)
@@ -3,4 +3,5 @@
 	<xacro:macro name="mobilebase" params="prefix='' name='mobilebase' suffix=''">
 		<link name="${prefix}${name}${suffix}_"></link>
+		<xacro:include filename="$(find transbot_description)/urdf/shelf_lifter/mobilebase/__extras__.urdf.xacro"></xacro:include>
 		<xacro:include filename="$(find transbot_description)/urdf/shelf_lifter/mobilebase/chassis.urdf.xacro"></xacro:include>
 		<xacro:include filename="$(find transbot_description)/urdf/shelf_lifter/mobilebase/control.urdf.xacro"></xacro:include>
@@ -38,4 +39,5 @@
 			<limit lower="0.0" upper="0.5" effort="1000000.0" velocity="1000000.0"></limit>
 		</joint>
+		<xacro:mobilebase-extras-description prefix="${prefix}${name}${suffix}"></xacro:mobilebase-extras-description>
 		<xacro:chassis prefix="${prefix}${name}${suffix}" suffix=""></xacro:chassis>
 		<xacro:control prefix="${prefix}${name}${suffix}" suffix=""></xacro:control>

File: robotics/transbot-ros2ws/src/transbot_description/urdf/shelf_lifter/shelf_lifter.urdf.xacro (robot description, xacro)
@@ -3,6 +3,10 @@
 	<xacro:macro name="shelf_lifter" params="prefix='' name='shelf_lifter' suffix=''">
 		<link name="${prefix}${name}${suffix}_"></link>
+		<xacro:include filename="$(find transbot_description)/urdf/shelf_lifter//__extras__.urdf.xacro"></xacro:include>
 		<xacro:include filename="$(find transbot_description)/urdf/shelf_lifter/mobilebase/mobilebase.urdf.xacro"></xacro:include>
 		<xacro:include filename="$(find transbot_description)/urdf/shelf_lifter/lifter.urdf.xacro"></xacro:include>
+		<xacro:include filename="$(find transbot_description)/urdf/shelf_lifter/camera.urdf.xacro"></xacro:include>
+		<xacro:include filename="$(find transbot_description)/urdf/shelf_lifter/lidar.urdf.xacro"></xacro:include>
+		<xacro:include filename="$(find transbot_description)/urdf/shelf_lifter/imu.urdf.xacro"></xacro:include>
 		<joint name="j/${prefix}${name}${suffix}mobilebase/_" type="fixed">
 			<origin xyz="0.0 0.0 0.0" rpy="0.0 0.0 0.0"></origin>
@@ -17,6 +21,25 @@
 			<limit lower="-0.005" upper="0.1" effort="1000000.0" velocity="1000000.0"></limit>
 		</joint>
+		<joint name="j/${prefix}${name}${suffix}camera" type="fixed">
+			<origin xyz="-0.375 0.0 0.6" rpy="0.0 0.08726646259971647 0.0"></origin>
+			<parent link="${prefix}${name}${suffix}_"></parent>
+			<child link="${prefix}${name}${suffix}camera"></child>
+		</joint>
+		<joint name="j/${prefix}${name}${suffix}lidar" type="fixed">
+			<origin xyz="0.275 0.0 0.18" rpy="0.0 0.0 0.0"></origin>
+			<parent link="${prefix}${name}${suffix}_"></parent>
+			<child link="${prefix}${name}${suffix}lidar"></child>
+		</joint>
+		<joint name="j/${prefix}${name}${suffix}imu" type="fixed">
+			<origin xyz="0.275 -0.25 0.18" rpy="0.0 0.0 0.0"></origin>
+			<parent link="${prefix}${name}${suffix}_"></parent>
+			<child link="${prefix}${name}${suffix}imu"></child>
+		</joint>
+		<xacro:shelf_lifter-extras-description prefix="${prefix}${name}${suffix}"></xacro:shelf_lifter-extras-description>
 		<xacro:mobilebase prefix="${prefix}${name}${suffix}" suffix="/"></xacro:mobilebase>
 		<xacro:lifter prefix="${prefix}${name}${suffix}" suffix=""></xacro:lifter>
+		<xacro:camera prefix="${prefix}${name}${suffix}" suffix=""></xacro:camera>
+		<xacro:lidar prefix="${prefix}${name}${suffix}" suffix=""></xacro:lidar>
+		<xacro:imu prefix="${prefix}${name}${suffix}" suffix=""></xacro:imu>
 	</xacro:macro>
 </robot>

File: robotics/transbot-ros2ws/src/transbot_gazebo/urdf/shelf_lifter/__all__.urdf.xacro (robot description, xacro)
@@ -11,5 +11,4 @@
 	<xacro:include filename="$(find transbot_description)/urdf/shelf_lifter/__all__.urdf.xacro"></xacro:include>
 	<xacro:include filename="$(find transbot_gazebo)/urdf/shelf_lifter/shelf_lifter.urdf.xacro"></xacro:include>
-	<xacro:include filename="$(find transbot_gazebo)/urdf/shelf_lifter/__extras__.urdf.xacro"></xacro:include>
 	<gazebo>
 		<plugin filename="gz_ros2_control-system" name="gz_ros2_control::GazeboSimROS2ControlPlugin">

File: robotics/transbot-ros2ws/src/transbot_gazebo/urdf/shelf_lifter/__extras__.urdf.xacro (robot description, xacro)
@@ -1,2 +1,25 @@
 <?xml version="1.0" encoding="utf-8"?>
-<robot xmlns:xacro="http://www.ros.org/wiki/xacro" name="shelf_lifter"></robot>
+<robot xmlns:xacro="http://www.ros.org/wiki/xacro" name="shelf_lifter">
+	<xacro:macro name="shelf_lifter-extras-gazebo" params="prefix='' name='shelf_lifter' suffix=''">
+		<gazebo reference="${prefix}${name}${prefix}camera">
+			<sensor name="camera" type="camera">
+				<always_on>true</always_on>
+				<update_rate>30</update_rate>
+				<topic>model/$(arg robot_name)/camera/image_raw</topic>
+				<gz_frame_id>${prefix}${name}${prefix}camera</gz_frame_id>
+				<camera>
+					<horizontal_fov>2</horizontal_fov>
+					<image>
+						<width>640</width>
+						<height>480</height>
+					<format>R8G8B8</format>
+					</image>
+					<clip>
+						<near>0.05</near>
+						<far>50</far>
+					</clip>
+				</camera>
+			</sensor>
+		</gazebo>
+	</xacro:macro>
+</robot>

File: robotics/transbot-ros2ws/src/transbot_gazebo/urdf/shelf_lifter/lifter.urdf.xacro (robot description, xacro)
@@ -3,3 +3,4 @@
 	<xacro:macro name="lifter-ros2_control_gazebo" params="prefix='' name='lifter' suffix=''"></xacro:macro>
 	<xacro:macro name="lifter-gz_reference" params="prefix='' name='lifter' suffix=''"></xacro:macro>
+	<xacro:lifter-extras-gazebo prefix="" name=""></xacro:lifter-extras-gazebo>
 </robot>

File: robotics/transbot-ros2ws/src/transbot_gazebo/urdf/shelf_lifter/mobilebase/__all__.urdf.xacro (robot description, xacro)
@@ -11,5 +11,4 @@
 	<xacro:include filename="$(find transbot_description)/urdf/shelf_lifter/__all__.urdf.xacro"></xacro:include>
 	<xacro:include filename="$(find transbot_gazebo)/urdf/shelf_lifter/mobilebase.urdf.xacro"></xacro:include>
-	<xacro:include filename="$(find transbot_gazebo)/urdf/shelf_lifter/__extras__.urdf.xacro"></xacro:include>
 	<gazebo>
 		<plugin filename="gz_ros2_control-system" name="gz_ros2_control::GazeboSimROS2ControlPlugin">

File: robotics/transbot-ros2ws/src/transbot_gazebo/urdf/shelf_lifter/mobilebase/__extras__.urdf.xacro (robot description, xacro)
@@ -1,2 +1,4 @@
 <?xml version="1.0" encoding="utf-8"?>
-<robot xmlns:xacro="http://www.ros.org/wiki/xacro" name="mobilebase"></robot>
+<robot xmlns:xacro="http://www.ros.org/wiki/xacro" name="mobilebase">
+	<xacro:macro name="mobilebase-extras-gazebo" params="prefix='' name='mobilebase' suffix=''"></xacro:macro>
+</robot>

File: robotics/transbot-ros2ws/src/transbot_gazebo/urdf/shelf_lifter/mobilebase/castor/__all__.urdf.xacro (robot description, xacro)
@@ -11,5 +11,4 @@
 	<xacro:include filename="$(find transbot_description)/urdf/shelf_lifter/mobilebase/__all__.urdf.xacro"></xacro:include>
 	<xacro:include filename="$(find transbot_gazebo)/urdf/shelf_lifter/mobilebase/castor.urdf.xacro"></xacro:include>
-	<xacro:include filename="$(find transbot_gazebo)/urdf/shelf_lifter/mobilebase/__extras__.urdf.xacro"></xacro:include>
 	<gazebo>
 		<plugin filename="gz_ros2_control-system" name="gz_ros2_control::GazeboSimROS2ControlPlugin">

File: robotics/transbot-ros2ws/src/transbot_gazebo/urdf/shelf_lifter/mobilebase/castor/castor.urdf.xacro (robot description, xacro)
@@ -1,4 +1,5 @@
 <?xml version="1.0" encoding="utf-8"?>
 <robot xmlns:xacro="http://www.ros.org/wiki/xacro" name="castor">
+	<xacro:include filename="$(find transbot_gazebo)/urdf/shelf_lifter/mobilebase/castor/__extras__.urdf.xacro"></xacro:include>
 	<xacro:macro name="castor-ros2_control_gazebo" params="prefix='' name='castor' suffix=''">
 		<joint name="j/${prefix}${name}${suffix}arm">
@@ -18,3 +19,4 @@
 	</xacro:macro>
 	<xacro:macro name="castor-gz_reference" params="prefix='' name='castor' suffix=''"></xacro:macro>
+	<xacro:castor-extras-gazebo prefix="" name=""></xacro:castor-extras-gazebo>
 </robot>
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