Commit message: fixed odometry offset for diff_drive_controller

File: robotics/transbot-ros2ws/src/transbot_description/urdf/shelf_lifter/mobilebase/__extras__.urdf.xacro (robot description, xacro)
@@ -1,4 +1,11 @@
 <?xml version="1.0" encoding="utf-8"?>
 <robot xmlns:xacro="http://www.ros.org/wiki/xacro" name="mobilebase">
-	<xacro:macro name="mobilebase-extras-description" params="prefix='' name='mobilebase' suffix=''"></xacro:macro>
+	<xacro:macro name="mobilebase-extras-description" params="prefix='' name='mobilebase' suffix=''">
+		<link name="drive_link"></link>
+		<joint name="j/drive_link" type="fixed">
+			<origin xyz="0.23 0.0 0.0" rpy="0.0 0.0 0.0"></origin>
+			<parent link="drive_link"></parent>
+			<child link="_"></child>
+		</joint>
+	</xacro:macro>
 </robot>
