Commit message: Depth cloud fixes

File: robotics/transbot-ros2ws/src/transbot_gazebo/urdf/shelf_lifter/__extras__.urdf.xacro (robot description, xacro)
@@ -2,10 +2,16 @@
 <robot xmlns:xacro="http://www.ros.org/wiki/xacro" name="shelf_lifter">
 	<xacro:macro name="shelf_lifter-extras-gazebo" params="prefix='' name='shelf_lifter' suffix=''">
+		<link name="${prefix}${name}${prefix}camera_optical_frame"/>
+		<joint name="j/${prefix}${name}${prefix}camera_optical_joint" type="fixed">
+			<parent link="${prefix}${name}${prefix}camera"/><child link="${prefix}${name}${prefix}camera_optical_frame"/>
+			<origin xyz="0 0 0" rpy="-1.5707963 0 -1.5707963"/>
+		</joint>
 		<gazebo reference="${prefix}${name}${prefix}camera">
 			<sensor name="camera" type="rgbd_camera">
+				<pose>0 0 0 0 0 0</pose>
 				<always_on>true</always_on>
 				<update_rate>10</update_rate>
 				<topic>model/$(arg robot_name)/rgbd_camera</topic>
-				<gz_frame_id>$(arg robot_name)/${prefix}${name}${prefix}camera</gz_frame_id>
+				<gz_frame_id>$(arg robot_name)/${prefix}${name}${prefix}camera_optical_frame</gz_frame_id>
 				<camera>
 					<horizontal_fov>1.396</horizontal_fov>
